Commit message: speed frac à l'arret + norm speed follower

File: corridor.urdf (robot description, URDF)
Before this commit: robot corridor, 5 links, 4 joints
Links:
- link wall_e: geometry collision box size=6.4 0.2 3.0; visual box size=6.4 0.2 3.0
- link wall_n: geometry collision box size=1.6 0.2 3.0; visual box size=1.6 0.2 3.0
- link wall_s: geometry collision box size=1.6 0.2 3.0; visual box size=1.6 0.2 3.0
- link wall_w: geometry collision box size=6.4 0.2 3.0; visual box size=6.4 0.2 3.0
Joints:
- joint wall_e_world: origin xyz=0.725 0 0 rpy=0 0 1.5707963267948966 -> xyz=0.85 0 0 rpy=0 0 1.5707963267948966
- joint wall_n_world: origin xyz=0 2.6 0 rpy=0 0 0 -> xyz=0 3.1 0 rpy=0 0 0
- joint wall_s_world: origin xyz=0 -2.6 0 rpy=0 0 0 -> xyz=0 -3.1 0 rpy=0 0 0
- joint wall_w_world: origin xyz=-0.725 0 0 rpy=0 0 1.5707963267948966 -> xyz=-0.85 0 0 rpy=0 0 1.5707963267948966
