Commit message: Modification pour être à la taille réel

File: Map/Multiple_corner/Multiple_corner.urdf (robot description, URDF)
Before this commit: robot corridor, 41 links, 40 joints
Links:
- added link Limit 1, mass 0; collision box size=0.04 4.6 1; visual box size=0.04 4.6 1
- added link Limit 2, mass 0; collision box size=0.04 4.6 1; visual box size=0.04 4.6 1
- added link Limit 3, mass 0; collision box size=0.04 3.4 1; visual box size=0.04 3.4 1
- added link Limit 4, mass 0; collision box size=0.04 3.4 1; visual box size=0.04 3.4 1
- link 10_left: geometry collision box size=0.04 0.5 0.5; visual box size=0.04 0.5 0.5
- link 10_right: geometry collision box size=0.04 0.5 0.5; visual box size=0.04 0.5 0.5
- link 11_left: geometry collision box size=0.04 0.5 0.5; visual box size=0.04 0.5 0.5
- link 11_right: geometry collision box size=0.04 0.5 0.5; visual box size=0.04 0.5 0.5
- link 12_left: geometry collision box size=0.04 0.5 0.5; visual box size=0.04 0.5 0.5
- link 12_right: geometry collision box size=0.04 0.5 0.5; visual box size=0.04 0.5 0.5
- link 13_front_down: geometry collision box size=0.04 0.0 0.5; visual box size=0.04 0.0 0.5
- link 13_front_up: geometry collision box size=0.04 0.5 0.5; visual box size=0.04 0.5 0.5
- link 13_left: geometry collision box size=0.04 0.0 0.5; visual box size=0.04 0.0 0.5
- link 13_right: geometry collision box size=0.04 0.5 0.5; visual box size=0.04 0.5 0.5
- link 14_front_down: geometry collision box size=0.04 0.0 0.5; visual box size=0.04 0.0 0.5
- link 14_front_up: geometry collision box size=0.04 0.5 0.5; visual box size=0.04 0.5 0.5
- link 14_left: geometry collision box size=0.04 0.0 0.5; visual box size=0.04 0.0 0.5
- link 14_right: geometry collision box size=0.04 0.5 0.5; visual box size=0.04 0.5 0.5
- link 1_left: geometry collision box size=0.04 0.5 0.5; visual box size=0.04 0.5 0.5
- link 1_right: geometry collision box size=0.04 0.5 0.5; visual box size=0.04 0.5 0.5
- link 2_front_down: geometry collision box size=0.04 0.0 0.5; visual box size=0.04 0.0 0.5
- link 2_front_up: geometry collision box size=0.04 0.5 0.5; visual box size=0.04 0.5 0.5
- link 2_left: geometry collision box size=0.04 0.0 0.5; visual box size=0.04 0.0 0.5
- link 2_right: geometry collision box size=0.04 0.5 0.5; visual box size=0.04 0.5 0.5
- link 3_left: geometry collision box size=0.04 0.5 0.5; visual box size=0.04 0.5 0.5
- link 3_right: geometry collision box size=0.04 0.5 0.5; visual box size=0.04 0.5 0.5
- link 4_front_down: geometry collision box size=0.04 0.0 0.5; visual box size=0.04 0.0 0.5
- link 4_front_up: geometry collision box size=0.04 0.5 0.5; visual box size=0.04 0.5 0.5
- link 4_left: geometry collision box size=0.04 0.0 0.5; visual box size=0.04 0.0 0.5
- link 4_right: geometry collision box size=0.04 0.5 0.5; visual box size=0.04 0.5 0.5
- link 5_left: geometry collision box size=0.04 0.5 0.5; visual box size=0.04 0.5 0.5
- link 5_right: geometry collision box size=0.04 0.5 0.5; visual box size=0.04 0.5 0.5
- link 6_front_down: geometry collision box size=0.04 0.0 0.5; visual box size=0.04 0.0 0.5
- link 6_front_up: geometry collision box size=0.04 0.5 0.5; visual box size=0.04 0.5 0.5
- link 6_left: geometry collision box size=0.04 0.0 0.5; visual box size=0.04 0.0 0.5
- link 6_right: geometry collision box size=0.04 0.5 0.5; visual box size=0.04 0.5 0.5
- link 7_left: geometry collision box size=0.04 0.5 0.5; visual box size=0.04 0.5 0.5
- link 7_right: geometry collision box size=0.04 0.5 0.5; visual box size=0.04 0.5 0.5
- link 8_left: geometry collision box size=0.04 0.5 0.5; visual box size=0.04 0.5 0.5
- link 8_right: geometry collision box size=0.04 0.5 0.5; visual box size=0.04 0.5 0.5
- link 9_front_down: geometry collision box size=0.04 0.0 0.5; visual box size=0.04 0.0 0.5
- link 9_front_up: geometry collision box size=0.04 0.5 0.5; visual box size=0.04 0.5 0.5
- link 9_left: geometry collision box size=0.04 0.0 0.5; visual box size=0.04 0.0 0.5
- link 9_right: geometry collision box size=0.04 0.5 0.5; visual box size=0.04 0.5 0.5
Joints:
- added joint Limit 1_world: type fixed, parent world, child Limit 1, origin xyz=1.7 0 0 rpy=0 0 0
- added joint Limit 2_world: type fixed, parent world, child Limit 2, origin xyz=-1.7 0 0 rpy=0 0 0
- added joint Limit 3_world: type fixed, parent world, child Limit 3, origin xyz=0 2.3 0 rpy=0 0 1.5707963267948966
- added joint Limit 4_world: type fixed, parent world, child Limit 4, origin xyz=0 -2.3 0 rpy=0 0 1.5707963267948966
- joint 10_left_world: origin xyz=-1.45 4.0 0 rpy=0 0 0 -> xyz=-0.22999999999999998 1.0 0 rpy=0 0 0
- joint 10_right_world: origin xyz=-2.55 4.0 0 rpy=0 0 0 -> xyz=-0.77 1.0 0 rpy=0 0 0
- joint 11_left_world: origin xyz=-1.45 2.0 0 rpy=0 0 0 -> xyz=-0.22999999999999998 0.5 0 rpy=0 0 0
- joint 11_right_world: origin xyz=-2.55 2.0 0 rpy=0 0 0 -> xyz=-0.77 0.5 0 rpy=0 0 0
- joint 12_left_world: origin xyz=-1.45 0.0 0 rpy=0 0 0 -> xyz=-0.22999999999999998 0.0 0 rpy=0 0 0
- joint 12_right_world: origin xyz=-2.55 0.0 0 rpy=0 0 0 -> xyz=-0.77 0.0 0 rpy=0 0 0
- joint 13_front_down_world: origin xyz=-1.45 -1.25 0 rpy=0 0 3.141592653589793 -> xyz=-0.22999999999999998 -0.25 0 rpy=0 0 3.141592653589793
- joint 13_front_up_world: origin xyz=-2.55 -1.75 0 rpy=0 0 3.141592653589793 -> xyz=-0.77 -0.5 0 rpy=0 0 3.141592653589793
- joint 13_left_world: origin xyz=-1.25 -1.45 0 rpy=0 0 1.5707963267948966 -> xyz=-0.25 -0.23 0 rpy=0 0 1.5707963267948966
- joint 13_right_world: origin xyz=-1.75 -2.55 0 rpy=0 0 1.5707963267948966 -> xyz=-0.5 -0.77 0 rpy=0 0 1.5707963267948966
- joint 14_front_down_world: origin xyz=-0.7499999999999999 -1.45 0 rpy=0 0 4.71238898038469 -> xyz=-0.24999999999999997 -0.22999999999999993 0 rpy=0 0 4.71238898038469
- joint 14_front_up_world: origin xyz=-0.25000000000000006 -2.55 0 rpy=0 0 4.71238898038469 -> xyz=-3.306546357697854e-17 -0.77 0 rpy=0 0 4.71238898038469
- joint 14_left_world: origin xyz=-0.5499999999999999 -1.25 0 rpy=0 0 3.141592653589793 -> xyz=-0.26999999999999996 -0.24999999999999994 0 rpy=0 0 3.141592653589793
- joint 14_right_world: origin xyz=0.55 -1.75 0 rpy=0 0 3.141592653589793 -> xyz=0.27 -0.5 0 rpy=0 0 3.141592653589793
- joint 1_left_world: origin xyz=0.55 0.0 0 rpy=0 0 0.0 -> xyz=0.27 0.0 0 rpy=0 0 0.0
- joint 1_right_world: origin xyz=-0.55 0.0 0 rpy=0 0 0.0 -> xyz=-0.27 0.0 0 rpy=0 0 0.0
- joint 2_front_down_world: origin xyz=0.75 1.45 0 rpy=0 0 1.5707963267948966 -> xyz=0.25 0.22999999999999998 0 rpy=0 0 1.5707963267948966
- joint 2_front_up_world: origin xyz=0.25 2.55 0 rpy=0 0 1.5707963267948966 -> xyz=0.0 0.77 0 rpy=0 0 1.5707963267948966
- joint 2_left_world: origin xyz=0.55 1.25 0 rpy=0 0 0.0 -> xyz=0.27 0.25 0 rpy=0 0 0.0
- joint 2_right_world: origin xyz=-0.55 1.75 0 rpy=0 0 0.0 -> xyz=-0.27 0.5 0 rpy=0 0 0.0
- joint 3_left_world: origin xyz=2.0 2.55 0 rpy=0 0 1.5707963267948966 -> xyz=0.5 0.77 0 rpy=0 0 1.5707963267948966
- joint 3_right_world: origin xyz=2.0 1.45 0 rpy=0 0 1.5707963267948966 -> xyz=0.5 0.22999999999999998 0 rpy=0 0 1.5707963267948966
- joint 4_front_down_world: origin xyz=3.25 2.55 0 rpy=0 0 4.71238898038469 -> xyz=0.75 0.77 0 rpy=0 0 4.71238898038469
- joint 4_front_up_world: origin xyz=3.75 1.45 0 rpy=0 0 4.71238898038469 -> xyz=1.0 0.22999999999999998 0 rpy=0 0 4.71238898038469
- joint 4_left_world: origin xyz=3.45 2.75 0 rpy=0 0 3.141592653589793 -> xyz=0.73 0.75 0 rpy=0 0 3.141592653589793
- joint 4_right_world: origin xyz=4.55 2.25 0 rpy=0 0 3.141592653589793 -> xyz=1.27 0.49999999999999994 0 rpy=0 0 3.141592653589793
- joint 5_left_world: origin xyz=4.55 4.0 0 rpy=0 0 0 -> xyz=1.27 1.0 0 rpy=0 0 0
- joint 5_right_world: origin xyz=3.45 4.0 0 rpy=0 0 0 -> xyz=0.73 1.0 0 rpy=0 0 0
- joint 6_front_down_world: origin xyz=3.45 5.25 0 rpy=0 0 6.283185307179586 -> xyz=0.73 1.25 0 rpy=0 0 6.283185307179586
- joint 6_front_up_world: origin xyz=4.55 5.75 0 rpy=0 0 6.283185307179586 -> xyz=1.27 1.5 0 rpy=0 0 6.283185307179586
- joint 6_left_world: origin xyz=3.25 5.45 0 rpy=0 0 4.71238898038469 -> xyz=0.75 1.23 0 rpy=0 0 4.71238898038469
- joint 6_right_world: origin xyz=3.75 6.55 0 rpy=0 0 4.71238898038469 -> xyz=1.0 1.77 0 rpy=0 0 4.71238898038469
- joint 7_left_world: origin xyz=2.0 6.55 0 rpy=0 0 1.5707963267948966 -> xyz=0.5 1.77 0 rpy=0 0 1.5707963267948966
- joint 7_right_world: origin xyz=2.0 5.45 0 rpy=0 0 1.5707963267948966 -> xyz=0.5 1.23 0 rpy=0 0 1.5707963267948966
- joint 8_left_world: origin xyz=3.367778697655222e-17 6.55 0 rpy=0 0 1.5707963267948966 -> xyz=1.653273178848927e-17 1.77 0 rpy=0 0 1.5707963267948966
- joint 8_right_world: origin xyz=-3.367778697655222e-17 5.45 0 rpy=0 0 1.5707963267948966 -> xyz=-1.653273178848927e-17 1.23 0 rpy=0 0 1.5707963267948966
- joint 9_front_down_world: origin xyz=-1.25 5.45 0 rpy=0 0 1.5707963267948966 -> xyz=-0.25 1.23 0 rpy=0 0 1.5707963267948966
- joint 9_front_up_world: origin xyz=-1.75 6.55 0 rpy=0 0 1.5707963267948966 -> xyz=-0.5 1.77 0 rpy=0 0 1.5707963267948966
- joint 9_left_world: origin xyz=-1.45 5.25 0 rpy=0 0 0 -> xyz=-0.22999999999999998 1.25 0 rpy=0 0 0
- joint 9_right_world: origin xyz=-2.55 5.75 0 rpy=0 0 0 -> xyz=-0.77 1.5 0 rpy=0 0 0

File: Map/Multiple_corner/Multiple_corner.xacro (robot description, xacro)
@@ -201,4 +201,41 @@
       rgba="${rgba}"/>
   </xacro:macro>
+  <!-- Map limit -->
+  <xacro:wall
+      name="Limit 1"
+      x="1.70"
+      y="0"
+      yaw="0"
+      length="4.6"
+      thk="0.04"
+      height="1"
+      rgba="${color}"/>
+  <xacro:wall
+      name="Limit 2"
+      x="-1.70"
+      y="0"
+      yaw="0"
+      length="4.6"
+      thk="0.04"
+      height="1"
+      rgba="${color}"/>
+  <xacro:wall
+      name="Limit 3"
+      x="0"
+      y="2.3"
+      yaw="${PI/2}"
+      length="3.4"
+      thk="0.04"
+      height="1"
+      rgba="${color}"/>
+  <xacro:wall
+      name="Limit 4"
+      x="0"
+      y="-2.3"
+      yaw="${PI/2}"
+      length="3.4"
+      thk="0.04"
+      height="1"
+      rgba="${color}"/>
   <!-- corridors (positionnés pour que l'intérieur fasse width) -->
   <xacro:corridor
@@ -215,5 +252,5 @@
   name="2"
   x="0.0"
-  y="2.0"
+  y="0.5"
   yaw="0.0"
   length="${L}"
@@ -224,6 +261,6 @@
   <xacro:corridor
   name="3"
-  x="2.0"
-  y="2.0"
+  x="0.5"
+  y="0.5"
   yaw="${PI/2}"
   length="${L}"
@@ -234,6 +271,6 @@
   <xacro:corner
   name="4"
-  x="4.0"
-  y="2.0"
+  x="1"
+  y="0.5"
   yaw="${PI}"
   length="${L}"
@@ -244,6 +281,6 @@
   <xacro:corridor
   name="5"
-  x="4.0"
-  y="4.0"
+  x="1"
+  y="1"
   yaw="${0}"
   length="${L}"
@@ -254,6 +291,6 @@
   <xacro:corner
   name="6"
-  x="4.0"
-  y="6.0"
+  x="1"
+  y="1.5"
   yaw="${PI*3/2}"
   length="${L}"
@@ -264,6 +301,6 @@
   <xacro:corridor
   name="7"
-  x="2.0"
-  y="6.0"
+  x="0.5"
+  y="1.5"
   yaw="${PI/2}"
   length="${L}"
@@ -275,5 +312,5 @@
   name="8"
   x="0.0"
-  y="6.0"
+  y="1.5"
   yaw="${PI/2}"
   length="${L}"
@@ -284,6 +321,6 @@
   <xacro:corner
   name="9"
-  x="-2.0"
-  y="6.0"
+  x="-0.5"
+  y="1.5"
   yaw="${0}"
   length="${L}"
@@ -294,6 +331,6 @@
   <xacro:corridor
   name="10"
-  x="-2.0"
-  y="4.0"
+  x="-0.5"
+  y="1"
   yaw="${0}"
   length="${L}"
@@ -304,6 +341,6 @@
   <xacro:corridor
   name="11"
-  x="-2.0"
-  y="2.0"
+  x="-0.5"
+  y="0.5"
   yaw="${0}"
   length="${L}"
@@ -314,5 +351,5 @@
   <xacro:corridor
   name="12"
-  x="-2.0"
+  x="-0.5"
   y="0.0"
   yaw="${0}"
@@ -324,6 +361,6 @@
   <xacro:corner
   name="13"
-  x="-2.0"
-  y="-2.0"
+  x="-0.5"
+  y="-0.5"
   yaw="${PI/2}"
   length="${L}"
@@ -335,5 +372,5 @@
   name="14"
   x="0.0"
-  y="-2.0"
+  y="-0.5"
   yaw="${PI}"
   length="${L}"

Commit message: Rotation carte multiplecorner, LeaderDeadEnd mais problème avec double virage, fix orchestrateur, mais passer par le send setpoint velocity world, + ajout d'un loger avec les positions du drone

File: Map/Multiple_corner/Multiple_corner.urdf (robot description, URDF)
Before this commit: robot corridor, 45 links, 44 joints
Links:
- link Limit 1: geometry collision box size=0.04 3.4 1; visual box size=0.04 3.4 1
- link Limit 2: geometry collision box size=0.04 3.4 1; visual box size=0.04 3.4 1
- link Limit 3: geometry collision box size=0.04 4.6 1; visual box size=0.04 4.6 1
- link Limit 4: geometry collision box size=0.04 4.6 1; visual box size=0.04 4.6 1
Joints:
- joint 10_left_world: origin xyz=-0.22999999999999998 1.0 0 rpy=0 0 0 -> xyz=-0.5 -0.22999999999999998 0 rpy=0 0 1.5707963267948966
- joint 10_right_world: origin xyz=-0.77 1.0 0 rpy=0 0 0 -> xyz=-0.5 -0.77 0 rpy=0 0 1.5707963267948966
- joint 11_left_world: origin xyz=-0.22999999999999998 0.5 0 rpy=0 0 0 -> xyz=1.653273178848927e-17 -0.22999999999999998 0 rpy=0 0 1.5707963267948966
- joint 11_right_world: origin xyz=-0.77 0.5 0 rpy=0 0 0 -> xyz=-1.653273178848927e-17 -0.77 0 rpy=0 0 1.5707963267948966
- joint 12_left_world: origin xyz=-0.22999999999999998 0.0 0 rpy=0 0 0 -> xyz=0.5 -0.22999999999999998 0 rpy=0 0 1.5707963267948966
- joint 12_right_world: origin xyz=-0.77 0.0 0 rpy=0 0 0 -> xyz=0.5 -0.77 0 rpy=0 0 1.5707963267948966
- joint 13_front_down_world: origin xyz=-0.22999999999999998 -0.25 0 rpy=0 0 3.141592653589793 -> xyz=0.75 -0.22999999999999993 0 rpy=0 0 4.71238898038469
- joint 13_front_up_world: origin xyz=-0.77 -0.5 0 rpy=0 0 3.141592653589793 -> xyz=1.0 -0.77 0 rpy=0 0 4.71238898038469
- joint 13_left_world: origin xyz=-0.25 -0.23 0 rpy=0 0 1.5707963267948966 -> xyz=0.73 -0.24999999999999994 0 rpy=0 0 3.141592653589793
- joint 13_right_world: origin xyz=-0.5 -0.77 0 rpy=0 0 1.5707963267948966 -> xyz=1.27 -0.5 0 rpy=0 0 3.141592653589793
- joint 14_front_down_world: origin xyz=-0.24999999999999997 -0.22999999999999993 0 rpy=0 0 4.71238898038469 -> xyz=0.73 -0.24999999999999994 0 rpy=0 0 6.283185307179586
- joint 14_front_up_world: origin xyz=-3.306546357697854e-17 -0.77 0 rpy=0 0 4.71238898038469 -> xyz=1.27 -4.9598195365467806e-17 0 rpy=0 0 6.283185307179586
- joint 14_left_world: origin xyz=-0.26999999999999996 -0.24999999999999994 0 rpy=0 0 3.141592653589793 -> xyz=0.75 -0.26999999999999996 0 rpy=0 0 4.71238898038469
- joint 14_right_world: origin xyz=0.27 -0.5 0 rpy=0 0 3.141592653589793 -> xyz=1.0 0.27 0 rpy=0 0 4.71238898038469
- joint 1_left_world: origin xyz=0.27 0.0 0 rpy=0 0 0.0 -> xyz=0.5 0.27 0 rpy=0 0 1.5707963267948966
- joint 1_right_world: origin xyz=-0.27 0.0 0 rpy=0 0 0.0 -> xyz=0.5 -0.27 0 rpy=0 0 1.5707963267948966
- joint 2_front_down_world: origin xyz=0.25 0.22999999999999998 0 rpy=0 0 1.5707963267948966 -> xyz=0.27 0.24999999999999997 0 rpy=0 0 3.141592653589793
- joint 2_front_up_world: origin xyz=0.0 0.77 0 rpy=0 0 1.5707963267948966 -> xyz=-0.27 1.653273178848927e-17 0 rpy=0 0 3.141592653589793
- joint 2_left_world: origin xyz=0.27 0.25 0 rpy=0 0 0.0 -> xyz=0.25 0.27 0 rpy=0 0 1.5707963267948966
- joint 2_right_world: origin xyz=-0.27 0.5 0 rpy=0 0 0.0 -> xyz=-1.653273178848927e-17 -0.27 0 rpy=0 0 1.5707963267948966
- joint 3_left_world: origin xyz=0.5 0.77 0 rpy=0 0 1.5707963267948966 -> xyz=0.27 0.5 0 rpy=0 0 0
- joint 3_right_world: origin xyz=0.5 0.22999999999999998 0 rpy=0 0 1.5707963267948966 -> xyz=-0.27 0.5 0 rpy=0 0 0
- joint 4_front_down_world: origin xyz=0.75 0.77 0 rpy=0 0 4.71238898038469 -> xyz=-0.2700000000000001 0.75 0 rpy=0 0 6.283185307179586
- joint 4_front_up_world: origin xyz=1.0 0.22999999999999998 0 rpy=0 0 4.71238898038469 -> xyz=0.27 1.0 0 rpy=0 0 6.283185307179586
- joint 4_left_world: origin xyz=0.73 0.75 0 rpy=0 0 3.141592653589793 -> xyz=-0.25000000000000006 0.73 0 rpy=0 0 4.71238898038469
- joint 4_right_world: origin xyz=1.27 0.49999999999999994 0 rpy=0 0 3.141592653589793 -> xyz=4.9598195365467806e-17 1.27 0 rpy=0 0 4.71238898038469
- joint 5_left_world: origin xyz=1.27 1.0 0 rpy=0 0 0 -> xyz=-0.5 1.27 0 rpy=0 0 1.5707963267948966
- joint 5_right_world: origin xyz=0.73 1.0 0 rpy=0 0 0 -> xyz=-0.5 0.73 0 rpy=0 0 1.5707963267948966
- joint 6_front_down_world: origin xyz=0.73 1.25 0 rpy=0 0 6.283185307179586 -> xyz=-0.75 0.73 0 rpy=0 0 1.5707963267948966
- joint 6_front_up_world: origin xyz=1.27 1.5 0 rpy=0 0 6.283185307179586 -> xyz=-1.0 1.27 0 rpy=0 0 1.5707963267948966
- joint 6_left_world: origin xyz=0.75 1.23 0 rpy=0 0 4.71238898038469 -> xyz=-0.73 0.75 0 rpy=0 0 0
- joint 6_right_world: origin xyz=1.0 1.77 0 rpy=0 0 4.71238898038469 -> xyz=-1.27 1.0 0 rpy=0 0 0
- joint 7_left_world: origin xyz=0.5 1.77 0 rpy=0 0 1.5707963267948966 -> xyz=-0.73 0.5 0 rpy=0 0 0
- joint 7_right_world: origin xyz=0.5 1.23 0 rpy=0 0 1.5707963267948966 -> xyz=-1.27 0.5 0 rpy=0 0 0
- joint 8_left_world: origin xyz=1.653273178848927e-17 1.77 0 rpy=0 0 1.5707963267948966 -> xyz=-0.73 0.0 0 rpy=0 0 0
- joint 8_right_world: origin xyz=-1.653273178848927e-17 1.23 0 rpy=0 0 1.5707963267948966 -> xyz=-1.27 0.0 0 rpy=0 0 0
- joint 9_front_down_world: origin xyz=-0.25 1.23 0 rpy=0 0 1.5707963267948966 -> xyz=-0.73 -0.25 0 rpy=0 0 3.141592653589793
- joint 9_front_up_world: origin xyz=-0.5 1.77 0 rpy=0 0 1.5707963267948966 -> xyz=-1.27 -0.5 0 rpy=0 0 3.141592653589793
- joint 9_left_world: origin xyz=-0.22999999999999998 1.25 0 rpy=0 0 0 -> xyz=-0.75 -0.23 0 rpy=0 0 1.5707963267948966
- joint 9_right_world: origin xyz=-0.77 1.5 0 rpy=0 0 0 -> xyz=-1.0 -0.77 0 rpy=0 0 1.5707963267948966
- joint Limit 1_world: origin xyz=1.7 0 0 rpy=0 0 0 -> xyz=2.3 0 0 rpy=0 0 0
- joint Limit 2_world: origin xyz=-1.7 0 0 rpy=0 0 0 -> xyz=-2.3 0 0 rpy=0 0 0
- joint Limit 3_world: origin xyz=0 2.3 0 rpy=0 0 1.5707963267948966 -> xyz=0 1.7 0 rpy=0 0 1.5707963267948966
- joint Limit 4_world: origin xyz=0 -2.3 0 rpy=0 0 1.5707963267948966 -> xyz=0 -1.7 0 rpy=0 0 1.5707963267948966

File: Map/Multiple_corner/Multiple_corner.xacro (robot description, xacro)
@@ -204,8 +204,8 @@
   <xacro:wall
       name="Limit 1"
-      x="1.70"
+      x="2.3"
       y="0"
       yaw="0"
-      length="4.6"
+      length="3.4"
       thk="0.04"
       height="1"
@@ -213,8 +213,8 @@
   <xacro:wall
       name="Limit 2"
-      x="-1.70"
+      x="-2.3"
       y="0"
       yaw="0"
-      length="4.6"
+      length="3.4"
       thk="0.04"
       height="1"
@@ -223,7 +223,7 @@
       name="Limit 3"
       x="0"
-      y="2.3"
+      y="1.70"
       yaw="${PI/2}"
-      length="3.4"
+      length="4.6"
       thk="0.04"
       height="1"
@@ -232,7 +232,7 @@
       name="Limit 4"
       x="0"
-      y="-2.3"
+      y="-1.70"
       yaw="${PI/2}"
-      length="3.4"
+      length="4.6"
       thk="0.04"
       height="1"
@@ -241,27 +241,27 @@
   <xacro:corridor
   name="1"
+  x="0.5"
+  y="0.0"
+  yaw="${PI/2}"
+  length="${L}"
+  width="${W}"
+  height="${H}"
+  thk="${thk}"
+  rgba="${color}"/>
+  <xacro:corner
+  name="2"
   x="0.0"
   y="0.0"
-  yaw="0.0"
-  length="${L}"
-  width="${W}"
-  height="${H}"
-  thk="${thk}"
-  rgba="${color}"/>
-  <xacro:corner
-  name="2"
-  x="0.0"
+  yaw="${PI/2}"
+  length="${L}"
+  width="${W}"
+  height="${H}"
+  thk="${thk}"
+  rgba="${color}"/>
+  <xacro:corridor
+  name="3"
+  x="0"
   y="0.5"
-  yaw="0.0"
-  length="${L}"
-  width="${W}"
-  height="${H}"
-  thk="${thk}"
-  rgba="${color}"/>
-  <xacro:corridor
-  name="3"
-  x="0.5"
-  y="0.5"
-  yaw="${PI/2}"
+  yaw="0"
   length="${L}"
   width="${W}"
@@ -271,7 +271,7 @@
   <xacro:corner
   name="4"
-  x="1"
-  y="0.5"
-  yaw="${PI}"
+  x="0"
+  y="1"
+  yaw="${3*PI/2}"
   length="${L}"
   width="${W}"
@@ -281,5 +281,15 @@
   <xacro:corridor
   name="5"
-  x="1"
+  x="-0.5"
+  y="1"
+  yaw="${PI/2}"
+  length="${L}"
+  width="${W}"
+  height="${H}"
+  thk="${thk}"
+  rgba="${color}"/>
+  <xacro:corner
+  name="6"
+  x="-1"
   y="1"
   yaw="${0}"
@@ -289,19 +299,9 @@
   thk="${thk}"
   rgba="${color}"/>
-  <xacro:corner
-  name="6"
-  x="1"
-  y="1.5"
-  yaw="${PI*3/2}"
-  length="${L}"
-  width="${W}"
-  height="${H}"
-  thk="${thk}"
-  rgba="${color}"/>
   <xacro:corridor
   name="7"
-  x="0.5"
-  y="1.5"
-  yaw="${PI/2}"
+  x="-1"
+  y="0.5"
+  yaw="${0}"
   length="${L}"
   width="${W}"
@@ -311,7 +311,7 @@
   <xacro:corridor
   name="8"
-  x="0.0"
-  y="1.5"
-  yaw="${PI/2}"
+  x="-1"
+  y="0"
+  yaw="${0}"
   length="${L}"
   width="${W}"
@@ -321,7 +321,7 @@
   <xacro:corner
   name="9"
-  x="-0.5"
-  y="1.5"
-  yaw="${0}"
+  x="-1"
+  y="-0.5"
+  yaw="${PI/2}"
   length="${L}"
   width="${W}"
@@ -332,6 +332,6 @@
   name="10"
   x="-0.5"
-  y="1"
-  yaw="${0}"
+  y="-0.5"
+  yaw="${PI/2}"
   length="${L}"
   width="${W}"
@@ -341,7 +341,7 @@
   <xacro:corridor
   name="11"
-  x="-0.5"
-  y="0.5"
-  yaw="${0}"
+  x="0"
+  y="-0.5"
+  yaw="${PI/2}"
   length="${L}"
   width="${W}"
@@ -351,7 +351,7 @@
   <xacro:corridor
   name="12"
-  x="-0.5"
-  y="0.0"
-  yaw="${0}"
+  x="0.5"
+  y="-0.5"
+  yaw="${PI/2}"
   length="${L}"
   width="${W}"
@@ -361,7 +361,7 @@
   <xacro:corner
   name="13"
-  x="-0.5"
-  y="-0.5"
-  yaw="${PI/2}"
+  x="1"
+  y="-0.5"
+  yaw="${PI}"
   length="${L}"
   width="${W}"
@@ -371,7 +371,7 @@
   <xacro:corner
   name="14"
-  x="0.0"
-  y="-0.5"
-  yaw="${PI}"
+  x="1"
+  y="0"
+  yaw="${3*PI/2}"
   length="${L}"
   width="${W}"
