Commit message: 2 drones intersection, petit bug avec le virage apres l'intersection, vérifier les variables 'global'

File: Map/Intersection/Intersection.urdf (robot description, URDF)
Before this commit: robot corridor, 35 links, 34 joints
Links:
- added link Limit 1, mass 0; collision box size=0.04 4.6 1; visual box size=0.04 4.6 1
- added link Limit 2, mass 0; collision box size=0.04 4.6 1; visual box size=0.04 4.6 1
- added link Limit 3, mass 0; collision box size=0.04 3.4 1; visual box size=0.04 3.4 1
- added link Limit 4, mass 0; collision box size=0.04 3.4 1; visual box size=0.04 3.4 1
- link 0_left: geometry collision box size=0.04 0.5 0.5; visual box size=0.04 0.5 0.5
- link 0_right: geometry collision box size=0.04 0.5 0.5; visual box size=0.04 0.5 0.5
- link 10_left: geometry collision box size=0.04 0.5 0.5; visual box size=0.04 0.5 0.5
- link 10_right: geometry collision box size=0.04 0.5 0.5; visual box size=0.04 0.5 0.5
- link 1_left: geometry collision box size=0.04 0.5 0.5; visual box size=0.04 0.5 0.5
- link 1_right: geometry collision box size=0.04 0.5 0.5; visual box size=0.04 0.5 0.5
- link 2_droit_h: geometry collision box size=0.04 0.0 0.5; visual box size=0.04 0.0 0.5
- link 2_droit_h_h: geometry collision box size=0.04 0.0 0.5; visual box size=0.04 0.0 0.5
- link 2_droit_v: geometry collision box size=0.04 0.0 0.5; visual box size=0.04 0.0 0.5
- link 2_droit_v_h: geometry collision box size=0.04 0.0 0.5; visual box size=0.04 0.0 0.5
- link 2_gauche_h: geometry collision box size=0.04 0.0 0.5; visual box size=0.04 0.0 0.5
- link 2_gauche_h_h: geometry collision box size=0.04 0.0 0.5; visual box size=0.04 0.0 0.5
- link 2_gauche_v: geometry collision box size=0.04 0.0 0.5; visual box size=0.04 0.0 0.5
- link 2_gauche_v_h: geometry collision box size=0.04 0.0 0.5; visual box size=0.04 0.0 0.5
- link 3_back: geometry collision box size=0.04 0.5 0.5; visual box size=0.04 0.5 0.5
- link 3_left: geometry collision box size=0.04 0.5 0.5; visual box size=0.04 0.5 0.5
- link 3_right: geometry collision box size=0.04 0.5 0.5; visual box size=0.04 0.5 0.5
- link 4_back: geometry collision box size=0.04 0.5 0.5; visual box size=0.04 0.5 0.5
- link 4_left: geometry collision box size=0.04 0.5 0.5; visual box size=0.04 0.5 0.5
- link 4_right: geometry collision box size=0.04 0.5 0.5; visual box size=0.04 0.5 0.5
- link 5_left: geometry collision box size=0.04 0.5 0.5; visual box size=0.04 0.5 0.5
- link 5_right: geometry collision box size=0.04 0.5 0.5; visual box size=0.04 0.5 0.5
- link 6_left: geometry collision box size=0.04 0.5 0.5; visual box size=0.04 0.5 0.5
- link 6_right: geometry collision box size=0.04 0.5 0.5; visual box size=0.04 0.5 0.5
- link 7_front_down: geometry collision box size=0.04 0.0 0.5; visual box size=0.04 0.0 0.5
- link 7_front_up: geometry collision box size=0.04 0.5 0.5; visual box size=0.04 0.5 0.5
- link 7_left: geometry collision box size=0.04 0.0 0.5; visual box size=0.04 0.0 0.5
- link 7_right: geometry collision box size=0.04 0.5 0.5; visual box size=0.04 0.5 0.5
- link 8_left: geometry collision box size=0.04 0.5 0.5; visual box size=0.04 0.5 0.5
- link 8_right: geometry collision box size=0.04 0.5 0.5; visual box size=0.04 0.5 0.5
- link 9_front_down: geometry collision box size=0.04 0.0 0.5; visual box size=0.04 0.0 0.5
- link 9_front_up: geometry collision box size=0.04 0.5 0.5; visual box size=0.04 0.5 0.5
- link 9_left: geometry collision box size=0.04 0.0 0.5; visual box size=0.04 0.0 0.5
- link 9_right: geometry collision box size=0.04 0.5 0.5; visual box size=0.04 0.5 0.5
Joints:
- added joint Limit 1_world: type fixed, parent world, child Limit 1, origin xyz=1.7 0 0 rpy=0 0 0
- added joint Limit 2_world: type fixed, parent world, child Limit 2, origin xyz=-1.7 0 0 rpy=0 0 0
- added joint Limit 3_world: type fixed, parent world, child Limit 3, origin xyz=0 2.3 0 rpy=0 0 1.5707963267948966
- added joint Limit 4_world: type fixed, parent world, child Limit 4, origin xyz=0 -2.3 0 rpy=0 0 1.5707963267948966
- joint 0_left_world: origin xyz=0.55 -2.0 0 rpy=0 0 0 -> xyz=0.77 -0.5 0 rpy=0 0 0
- joint 0_right_world: origin xyz=-0.55 -2.0 0 rpy=0 0 0 -> xyz=0.22999999999999998 -0.5 0 rpy=0 0 0
- joint 10_left_world: origin xyz=-8.0 6.55 0 rpy=0 0 1.5707963267948966 -> xyz=-1.5 1.77 0 rpy=0 0 1.5707963267948966
- joint 10_right_world: origin xyz=-8.0 5.45 0 rpy=0 0 1.5707963267948966 -> xyz=-1.5 1.23 0 rpy=0 0 1.5707963267948966
- joint 1_left_world: origin xyz=0.55 0.0 0 rpy=0 0 0 -> xyz=0.77 0.0 0 rpy=0 0 0
- joint 1_right_world: origin xyz=-0.55 0.0 0 rpy=0 0 0 -> xyz=0.22999999999999998 0.0 0 rpy=0 0 0
- joint 2_droit_h_h_world: origin xyz=-0.55 2.75 0 rpy=0 0 3.141592653589793 -> xyz=0.22999999999999998 0.75 0 rpy=0 0 3.141592653589793
- joint 2_droit_h_world: origin xyz=0.55 2.75 0 rpy=0 0 3.141592653589793 -> xyz=0.77 0.75 0 rpy=0 0 3.141592653589793
- joint 2_droit_v_h_world: origin xyz=-0.75 2.55 0 rpy=0 0 1.5707963267948966 -> xyz=0.25 0.77 0 rpy=0 0 1.5707963267948966
- joint 2_droit_v_world: origin xyz=0.75 2.55 0 rpy=0 0 1.5707963267948966 -> xyz=0.75 0.77 0 rpy=0 0 1.5707963267948966
- joint 2_gauche_h_h_world: origin xyz=-0.55 1.25 0 rpy=0 0 3.141592653589793 -> xyz=0.22999999999999998 0.25 0 rpy=0 0 3.141592653589793
- joint 2_gauche_h_world: origin xyz=0.55 1.25 0 rpy=0 0 3.141592653589793 -> xyz=0.77 0.24999999999999997 0 rpy=0 0 3.141592653589793
- joint 2_gauche_v_h_world: origin xyz=-0.75 1.45 0 rpy=0 0 1.5707963267948966 -> xyz=0.25 0.23 0 rpy=0 0 1.5707963267948966
- joint 2_gauche_v_world: origin xyz=0.75 1.45 0 rpy=0 0 1.5707963267948966 -> xyz=0.75 0.22999999999999995 0 rpy=0 0 1.5707963267948966
- joint 3_back_world: origin xyz=1.285879139104721e-16 5.05 0 rpy=0 0 4.71238898038469 -> xyz=0.5 1.27 0 rpy=0 0 4.71238898038469
- joint 3_left_world: origin xyz=-0.55 4.0 0 rpy=0 0 3.141592653589793 -> xyz=0.22999999999999998 1.0 0 rpy=0 0 3.141592653589793
- joint 3_right_world: origin xyz=0.55 4.0 0 rpy=0 0 3.141592653589793 -> xyz=0.77 1.0 0 rpy=0 0 3.141592653589793
- joint 4_back_world: origin xyz=3.05 2.0 0 rpy=0 0 3.141592653589793 -> xyz=1.27 0.5 0 rpy=0 0 3.141592653589793
- joint 4_left_world: origin xyz=2.0 2.55 0 rpy=0 0 1.5707963267948966 -> xyz=1.0 0.77 0 rpy=0 0 1.5707963267948966
- joint 4_right_world: origin xyz=2.0 1.45 0 rpy=0 0 1.5707963267948966 -> xyz=1.0 0.22999999999999998 0 rpy=0 0 1.5707963267948966
- joint 5_left_world: origin xyz=-2.0 1.45 0 rpy=0 0 4.71238898038469 -> xyz=-4.9598195365467806e-17 0.22999999999999998 0 rpy=0 0 4.71238898038469
- joint 5_right_world: origin xyz=-2.0 2.55 0 rpy=0 0 4.71238898038469 -> xyz=4.9598195365467806e-17 0.77 0 rpy=0 0 4.71238898038469
- joint 6_left_world: origin xyz=-4.0 1.45 0 rpy=0 0 4.71238898038469 -> xyz=-0.5 0.22999999999999998 0 rpy=0 0 4.71238898038469
- joint 6_right_world: origin xyz=-4.0 2.55 0 rpy=0 0 4.71238898038469 -> xyz=-0.49999999999999994 0.77 0 rpy=0 0 4.71238898038469
- joint 7_front_down_world: origin xyz=-5.45 2.75 0 rpy=0 0 3.141592653589793 -> xyz=-0.73 0.75 0 rpy=0 0 3.141592653589793
- joint 7_front_up_world: origin xyz=-6.55 2.25 0 rpy=0 0 3.141592653589793 -> xyz=-1.27 0.5 0 rpy=0 0 3.141592653589793
- joint 7_left_world: origin xyz=-5.25 2.55 0 rpy=0 0 1.5707963267948966 -> xyz=-0.75 0.77 0 rpy=0 0 1.5707963267948966
- joint 7_right_world: origin xyz=-5.75 1.45 0 rpy=0 0 1.5707963267948966 -> xyz=-1.0 0.22999999999999998 0 rpy=0 0 1.5707963267948966
- joint 8_left_world: origin xyz=-5.45 4.0 0 rpy=0 0 0 -> xyz=-0.73 1.0 0 rpy=0 0 0
- joint 8_right_world: origin xyz=-6.55 4.0 0 rpy=0 0 0 -> xyz=-1.27 1.0 0 rpy=0 0 0
- joint 9_front_down_world: origin xyz=-6.55 5.25 0 rpy=0 0 6.283185307179586 -> xyz=-1.27 1.25 0 rpy=0 0 6.283185307179586
- joint 9_front_up_world: origin xyz=-5.45 5.75 0 rpy=0 0 6.283185307179586 -> xyz=-0.73 1.5 0 rpy=0 0 6.283185307179586
- joint 9_left_world: origin xyz=-6.75 5.45 0 rpy=0 0 4.71238898038469 -> xyz=-1.25 1.23 0 rpy=0 0 4.71238898038469
- joint 9_right_world: origin xyz=-6.25 6.55 0 rpy=0 0 4.71238898038469 -> xyz=-1.0 1.77 0 rpy=0 0 4.71238898038469

File: Map/Intersection/Intersection.xacro (robot description, xacro)
@@ -410,9 +410,46 @@
       rgba="${rgba}" />
   </xacro:macro>
+  <!-- Map limit -->
+  <xacro:wall
+      name="Limit 1"
+      x="1.70"
+      y="0"
+      yaw="0"
+      length="4.6"
+      thk="0.04"
+      height="1"
+      rgba="${color}"/>
+  <xacro:wall
+      name="Limit 2"
+      x="-1.70"
+      y="0"
+      yaw="0"
+      length="4.6"
+      thk="0.04"
+      height="1"
+      rgba="${color}"/>
+  <xacro:wall
+      name="Limit 3"
+      x="0"
+      y="2.3"
+      yaw="${PI/2}"
+      length="3.4"
+      thk="0.04"
+      height="1"
+      rgba="${color}"/>
+  <xacro:wall
+      name="Limit 4"
+      x="0"
+      y="-2.3"
+      yaw="${PI/2}"
+      length="3.4"
+      thk="0.04"
+      height="1"
+      rgba="${color}"/>
   <!-- corridors (positionnés pour que l'intérieur fasse width) -->
   <xacro:corridor
   name="0"
-  x="0.0"
-  y="-2.0"
+  x="0.5"
+  y="-0.5"
   yaw="${0}"
   length="${L}"
@@ -423,5 +460,5 @@
   <xacro:corridor
   name="1"
-  x="0.0"
+  x="0.5"
   y="0.0"
   yaw="${0}"
@@ -433,6 +470,6 @@
   <xacro:C_intersection
   name="2"
-  x="0.0"
-  y="2.0"
+  x="0.5"
+  y="0.5"
   yaw="${PI/2}"
   length="${L}"
@@ -443,6 +480,6 @@
   <xacro:u_corridor
   name="3"
-  x="0.0"
-  y="4.0"
+  x="0.5"
+  y="1.0"
   yaw="${PI}"
   length="${L}"
@@ -453,6 +490,6 @@
   <xacro:u_corridor
   name="4"
-  x="2.0"
-  y="2.0"
+  x="1.0"
+  y="0.5"
   yaw="${PI/2}"
   length="${L}"
@@ -463,6 +500,6 @@
   <xacro:corridor
   name="5"
-  x="-2.0"
-  y="2.0"
+  x="0.0"
+  y="0.5"
   yaw="${PI*3/2}"
   length="${L}"
@@ -473,6 +510,6 @@
   <xacro:corridor
   name="6"
-  x="-4.0"
-  y="2.0"
+  x="-0.5"
+  y="0.5"
   yaw="${PI*3/2}"
   length="${L}"
@@ -483,6 +520,6 @@
   <xacro:corner
   name="7"
-  x="-6.0"
-  y="2.0"
+  x="-1.0"
+  y="0.5"
   yaw="${PI/2}"
   length="${L}"
@@ -493,6 +530,6 @@
     <xacro:corridor
   name="8"
-  x="-6.0"
-  y="4.0"
+  x="-1.0"
+  y="1.0"
   yaw="${0}"
   length="${L}"
@@ -503,6 +540,6 @@
   <xacro:corner
     name="9"
-    x="-6.0"
-    y="6.0"
+    x="-1.0"
+    y="1.5"
     yaw="${PI*3/2}"
     length="${L}"
@@ -513,6 +550,6 @@
   <xacro:corridor
     name="10"
-    x="-8.0"
-    y="6.0"
+    x="-1.5"
+    y="1.5"
     yaw="${pi/2}"
     length="${L}"

Commit message: Dead end, mais bug intersection avec beaucoup de drones

File: Map/Intersection/Intersection.urdf (robot description, URDF)
Before this commit: robot corridor, 39 links, 38 joints
Links:
- added link 11_left, mass 0; collision box size=0.04 0.5 0.5; visual box size=0.04 0.5 0.5
- added link 11_right, mass 0; collision box size=0.04 0.5 0.5; visual box size=0.04 0.5 0.5
- added link 12_left, mass 0; collision box size=0.04 0.5 0.5; visual box size=0.04 0.5 0.5
- added link 12_right, mass 0; collision box size=0.04 0.5 0.5; visual box size=0.04 0.5 0.5
- added link 13_left, mass 0; collision box size=0.04 0.5 0.5; visual box size=0.04 0.5 0.5
- added link 13_right, mass 0; collision box size=0.04 0.5 0.5; visual box size=0.04 0.5 0.5
- added link 14_left, mass 0; collision box size=0.04 0.5 0.5; visual box size=0.04 0.5 0.5
- added link 14_right, mass 0; collision box size=0.04 0.5 0.5; visual box size=0.04 0.5 0.5
Joints:
- added joint 11_left_world: type fixed, parent world, child 11_left, origin xyz=0.77 -0.5 0 rpy=0 0 0
- added joint 11_right_world: type fixed, parent world, child 11_right, origin xyz=0.22999999999999998 -0.5 0 rpy=0 0 0
- added joint 12_left_world: type fixed, parent world, child 12_left, origin xyz=0.77 -1.0 0 rpy=0 0 0
- added joint 12_right_world: type fixed, parent world, child 12_right, origin xyz=0.22999999999999998 -1.0 0 rpy=0 0 0
- added joint 13_left_world: type fixed, parent world, child 13_left, origin xyz=0.77 -1.5 0 rpy=0 0 0
- added joint 13_right_world: type fixed, parent world, child 13_right, origin xyz=0.22999999999999998 -1.5 0 rpy=0 0 0
- added joint 14_left_world: type fixed, parent world, child 14_left, origin xyz=0.77 -2.0 0 rpy=0 0 0
- added joint 14_right_world: type fixed, parent world, child 14_right, origin xyz=0.22999999999999998 -2.0 0 rpy=0 0 0

File: Map/Intersection/Intersection.xacro (robot description, xacro)
@@ -558,3 +558,43 @@
     thk="${thk}"
     rgba="${color}"/>
+  <xacro:corridor
+    name="11"
+    x="0.5"
+    y="-0.5"
+    yaw="${0}"
+    length="${L}"
+    width="${W}"
+    height="${H}"
+    thk="${thk}"
+    rgba="${color}"/>
+  <xacro:corridor
+    name="12"
+    x="0.5"
+    y="-1"
+    yaw="${0}"
+    length="${L}"
+    width="${W}"
+    height="${H}"
+    thk="${thk}"
+    rgba="${color}"/>
+  <xacro:corridor
+    name="13"
+    x="0.5"
+    y="-1.5"
+    yaw="${0}"
+    length="${L}"
+    width="${W}"
+    height="${H}"
+    thk="${thk}"
+    rgba="${color}"/>
+  <xacro:corridor
+    name="14"
+    x="0.5"
+    y="-2"
+    yaw="${0}"
+    length="${L}"
+    width="${W}"
+    height="${H}"
+    thk="${thk}"
+    rgba="${color}"/>
 </robot>
