Commit message: Rotation carte intersection

File: Map/Intersection/Intersection.urdf (robot description, URDF)
Before this commit: robot corridor, 47 links, 46 joints
Links:
- removed link 13_left
- removed link 13_right
- removed link 14_left
- removed link 14_right
- removed link 2_droit_h
- removed link 2_droit_h_h
- removed link 2_droit_v
- removed link 2_droit_v_h
- removed link 2_gauche_h
- removed link 2_gauche_h_h
- removed link 2_gauche_v
- removed link 2_gauche_v_h
- removed link 3_back
- removed link 4_back
- removed link 4_left
- removed link 4_right
- removed link 7_front_down
- removed link 7_front_up
- added link 11_front_down, mass 0; collision box size=0.04 0.0 0.5; visual box size=0.04 0.0 0.5
- added link 11_front_up, mass 0; collision box size=0.04 0.5 0.5; visual box size=0.04 0.5 0.5
- added link 2_left, mass 0; collision box size=0.04 0.5 0.5; visual box size=0.04 0.5 0.5
- added link 2_right, mass 0; collision box size=0.04 0.5 0.5; visual box size=0.04 0.5 0.5
- added link 4_droit_h, mass 0; collision box size=0.04 0.0 0.5; visual box size=0.04 0.0 0.5
- added link 4_droit_h_h, mass 0; collision box size=0.04 0.0 0.5; visual box size=0.04 0.0 0.5
- added link 4_droit_v, mass 0; collision box size=0.04 0.0 0.5; visual box size=0.04 0.0 0.5
- added link 4_droit_v_h, mass 0; collision box size=0.04 0.0 0.5; visual box size=0.04 0.0 0.5
- added link 4_gauche_h, mass 0; collision box size=0.04 0.0 0.5; visual box size=0.04 0.0 0.5
- added link 4_gauche_h_h, mass 0; collision box size=0.04 0.0 0.5; visual box size=0.04 0.0 0.5
- added link 4_gauche_v, mass 0; collision box size=0.04 0.0 0.5; visual box size=0.04 0.0 0.5
- added link 4_gauche_v_h, mass 0; collision box size=0.04 0.0 0.5; visual box size=0.04 0.0 0.5
- added link 5_back, mass 0; collision box size=0.04 0.5 0.5; visual box size=0.04 0.5 0.5
- added link 6_back, mass 0; collision box size=0.04 0.5 0.5; visual box size=0.04 0.5 0.5
- link 11_left: geometry collision box size=0.04 0.0 0.5; visual box size=0.04 0.0 0.5
- link 7_left: geometry collision box size=0.04 0.5 0.5; visual box size=0.04 0.5 0.5
- link Limit 1: geometry collision box size=0.04 3.4 1; visual box size=0.04 3.4 1
- link Limit 2: geometry collision box size=0.04 3.4 1; visual box size=0.04 3.4 1
- link Limit 3: geometry collision box size=0.04 4.6 1; visual box size=0.04 4.6 1
- link Limit 4: geometry collision box size=0.04 4.6 1; visual box size=0.04 4.6 1
Joints:
- removed joint 13_left_world
- removed joint 13_right_world
- removed joint 14_left_world
- removed joint 14_right_world
- removed joint 2_droit_h_h_world
- removed joint 2_droit_h_world
- removed joint 2_droit_v_h_world
- removed joint 2_droit_v_world
- removed joint 2_gauche_h_h_world
- removed joint 2_gauche_h_world
- removed joint 2_gauche_v_h_world
- removed joint 2_gauche_v_world
- removed joint 3_back_world
- removed joint 4_back_world
- removed joint 4_left_world
- removed joint 4_right_world
- removed joint 7_front_down_world
- removed joint 7_front_up_world
- added joint 11_front_down_world: type fixed, parent world, child 11_front_down, origin xyz=-0.75 -1.27 0 rpy=0 0 1.5707963267948966
- added joint 11_front_up_world: type fixed, parent world, child 11_front_up, origin xyz=-1.0 -0.73 0 rpy=0 0 1.5707963267948966
- added joint 2_left_world: type fixed, parent world, child 2_left, origin xyz=1.0 0.77 0 rpy=0 0 1.5707963267948966
- added joint 2_right_world: type fixed, parent world, child 2_right, origin xyz=1.0 0.22999999999999998 0 rpy=0 0 1.5707963267948966
- added joint 4_droit_h_h_world: type fixed, parent world, child 4_droit_h_h, origin xyz=0.25 0.77 0 rpy=0 0 1.5707963267948966
- added joint 4_droit_h_world: type fixed, parent world, child 4_droit_h, origin xyz=0.25 0.22999999999999998 0 rpy=0 0 1.5707963267948966
- added joint 4_droit_v_h_world: type fixed, parent world, child 4_droit_v_h, origin xyz=0.27 0.75 0 rpy=0 0 0
- added joint 4_droit_v_world: type fixed, parent world, child 4_droit_v, origin xyz=0.27 0.25 0 rpy=0 0 0
- added joint 4_gauche_h_h_world: type fixed, parent world, child 4_gauche_h_h, origin xyz=-0.25 0.77 0 rpy=0 0 1.5707963267948966
- added joint 4_gauche_h_world: type fixed, parent world, child 4_gauche_h, origin xyz=-0.25 0.22999999999999998 0 rpy=0 0 1.5707963267948966
- added joint 4_gauche_v_h_world: type fixed, parent world, child 4_gauche_v_h, origin xyz=-0.27 0.75 0 rpy=0 0 0
- added joint 4_gauche_v_world: type fixed, parent world, child 4_gauche_v, origin xyz=-0.27 0.25 0 rpy=0 0 0
- added joint 5_back_world: type fixed, parent world, child 5_back, origin xyz=-0.77 0.5 0 rpy=0 0 6.283185307179586
- added joint 6_back_world: type fixed, parent world, child 6_back, origin xyz=3.306546357697854e-17 1.27 0 rpy=0 0 4.71238898038469
- joint 0_left_world: origin xyz=0.77 -0.5 0 rpy=0 0 0 -> xyz=2.0 0.77 0 rpy=0 0 1.5707963267948966
- joint 0_right_world: origin xyz=0.22999999999999998 -0.5 0 rpy=0 0 0 -> xyz=2.0 0.22999999999999998 0 rpy=0 0 1.5707963267948966
- joint 10_left_world: origin xyz=-1.5 1.77 0 rpy=0 0 1.5707963267948966 -> xyz=-0.5 -0.73 0 rpy=0 0 1.5707963267948966
- joint 10_right_world: origin xyz=-1.5 1.23 0 rpy=0 0 1.5707963267948966 -> xyz=-0.5 -1.27 0 rpy=0 0 1.5707963267948966
- joint 11_left_world: origin xyz=0.77 -0.5 0 rpy=0 0 0 -> xyz=-0.73 -1.25 0 rpy=0 0 0
- joint 11_right_world: origin xyz=0.22999999999999998 -0.5 0 rpy=0 0 0 -> xyz=-1.27 -1.0 0 rpy=0 0 0
- joint 12_left_world: origin xyz=0.77 -1.0 0 rpy=0 0 0 -> xyz=-0.73 -1.5 0 rpy=0 0 0
- joint 12_right_world: origin xyz=0.22999999999999998 -1.0 0 rpy=0 0 0 -> xyz=-1.27 -1.5 0 rpy=0 0 0
- joint 1_left_world: origin xyz=0.77 0.0 0 rpy=0 0 0 -> xyz=1.5 0.77 0 rpy=0 0 1.5707963267948966
- joint 1_right_world: origin xyz=0.22999999999999998 0.0 0 rpy=0 0 0 -> xyz=1.5 0.22999999999999998 0 rpy=0 0 1.5707963267948966
- joint 3_left_world: origin xyz=0.22999999999999998 1.0 0 rpy=0 0 3.141592653589793 -> xyz=0.5 0.77 0 rpy=0 0 1.5707963267948966
- joint 3_right_world: origin xyz=0.77 1.0 0 rpy=0 0 3.141592653589793 -> xyz=0.5 0.22999999999999998 0 rpy=0 0 1.5707963267948966
- joint 5_left_world: origin xyz=-4.9598195365467806e-17 0.22999999999999998 0 rpy=0 0 4.71238898038469 -> xyz=-0.5 0.22999999999999998 0 rpy=0 0 4.71238898038469
- joint 5_right_world: origin xyz=4.9598195365467806e-17 0.77 0 rpy=0 0 4.71238898038469 -> xyz=-0.49999999999999994 0.77 0 rpy=0 0 4.71238898038469
- joint 6_left_world: origin xyz=-0.5 0.22999999999999998 0 rpy=0 0 4.71238898038469 -> xyz=-0.27 1.0 0 rpy=0 0 3.141592653589793
- joint 6_right_world: origin xyz=-0.49999999999999994 0.77 0 rpy=0 0 4.71238898038469 -> xyz=0.27 1.0 0 rpy=0 0 3.141592653589793
- joint 7_left_world: origin xyz=-0.75 0.77 0 rpy=0 0 1.5707963267948966 -> xyz=0.27 0.0 0 rpy=0 0 0
- joint 7_right_world: origin xyz=-1.0 0.22999999999999998 0 rpy=0 0 1.5707963267948966 -> xyz=-0.27 0.0 0 rpy=0 0 0
- joint 8_left_world: origin xyz=-0.73 1.0 0 rpy=0 0 0 -> xyz=0.27 -0.5 0 rpy=0 0 0
- joint 8_right_world: origin xyz=-1.27 1.0 0 rpy=0 0 0 -> xyz=-0.27 -0.5 0 rpy=0 0 0
- joint 9_front_down_world: origin xyz=-1.27 1.25 0 rpy=0 0 6.283185307179586 -> xyz=-0.24999999999999997 -0.73 0 rpy=0 0 4.71238898038469
- joint 9_front_up_world: origin xyz=-0.73 1.5 0 rpy=0 0 6.283185307179586 -> xyz=-3.306546357697854e-17 -1.27 0 rpy=0 0 4.71238898038469
- joint 9_left_world: origin xyz=-1.25 1.23 0 rpy=0 0 4.71238898038469 -> xyz=-0.26999999999999996 -0.75 0 rpy=0 0 3.141592653589793
- joint 9_right_world: origin xyz=-1.0 1.77 0 rpy=0 0 4.71238898038469 -> xyz=0.27 -1.0 0 rpy=0 0 3.141592653589793
- joint Limit 1_world: origin xyz=1.7 0 0 rpy=0 0 0 -> xyz=2.3 0 0 rpy=0 0 0
- joint Limit 2_world: origin xyz=-1.7 0 0 rpy=0 0 0 -> xyz=-2.3 0 0 rpy=0 0 0
- joint Limit 3_world: origin xyz=0 2.3 0 rpy=0 0 1.5707963267948966 -> xyz=0 1.7 0 rpy=0 0 1.5707963267948966
- joint Limit 4_world: origin xyz=0 -2.3 0 rpy=0 0 1.5707963267948966 -> xyz=0 -1.7 0 rpy=0 0 1.5707963267948966

File: Map/Intersection/Intersection.xacro (robot description, xacro)
@@ -413,8 +413,8 @@
   <xacro:wall
       name="Limit 1"
-      x="1.70"
+      x="2.3"
       y="0"
       yaw="0"
-      length="4.6"
+      length="3.4"
       thk="0.04"
       height="1"
@@ -422,8 +422,8 @@
   <xacro:wall
       name="Limit 2"
-      x="-1.70"
+      x="-2.3"
       y="0"
       yaw="0"
-      length="4.6"
+      length="3.4"
       thk="0.04"
       height="1"
@@ -432,7 +432,7 @@
       name="Limit 3"
       x="0"
-      y="2.3"
+      y="1.70"
       yaw="${PI/2}"
-      length="3.4"
+      length="4.6"
       thk="0.04"
       height="1"
@@ -441,7 +441,7 @@
       name="Limit 4"
       x="0"
-      y="-2.3"
+      y="-1.70"
       yaw="${PI/2}"
-      length="3.4"
+      length="4.6"
       thk="0.04"
       height="1"
@@ -450,25 +450,5 @@
   <xacro:corridor
   name="0"
-  x="0.5"
-  y="-0.5"
-  yaw="${0}"
-  length="${L}"
-  width="${W}"
-  height="${H}"
-  thk="${thk}"
-  rgba="${color}"/>
-  <xacro:corridor
-  name="1"
-  x="0.5"
-  y="0.0"
-  yaw="${0}"
-  length="${L}"
-  width="${W}"
-  height="${H}"
-  thk="${thk}"
-  rgba="${color}"/>
-  <xacro:C_intersection
-  name="2"
-  x="0.5"
+  x="2"
   y="0.5"
   yaw="${PI/2}"
@@ -478,17 +458,7 @@
   thk="${thk}"
   rgba="${color}"/>
-  <xacro:u_corridor
-  name="3"
-  x="0.5"
-  y="1.0"
-  yaw="${PI}"
-  length="${L}"
-  width="${W}"
-  height="${H}"
-  thk="${thk}"
-  rgba="${color}"/>
-  <xacro:u_corridor
-  name="4"
-  x="1.0"
+  <xacro:corridor
+  name="1"
+  x="1.5"
   y="0.5"
   yaw="${PI/2}"
@@ -499,26 +469,6 @@
   rgba="${color}"/>
   <xacro:corridor
-  name="5"
-  x="0.0"
-  y="0.5"
-  yaw="${PI*3/2}"
-  length="${L}"
-  width="${W}"
-  height="${H}"
-  thk="${thk}"
-  rgba="${color}"/>
-  <xacro:corridor
-  name="6"
-  x="-0.5"
-  y="0.5"
-  yaw="${PI*3/2}"
-  length="${L}"
-  width="${W}"
-  height="${H}"
-  thk="${thk}"
-  rgba="${color}"/>
-  <xacro:corner
-  name="7"
-  x="-1.0"
+  name="2"
+  x="1"
   y="0.5"
   yaw="${PI/2}"
@@ -528,8 +478,88 @@
   thk="${thk}"
   rgba="${color}"/>
-    <xacro:corridor
+  <xacro:corridor
+  name="3"
+  x=".5"
+  y="0.5"
+  yaw="${PI/2}"
+  length="${L}"
+  width="${W}"
+  height="${H}"
+  thk="${thk}"
+  rgba="${color}"/>
+  <xacro:C_intersection
+  name="4"
+  x="0"
+  y="0.5"
+  yaw="0"
+  length="${L}"
+  width="${W}"
+  height="${H}"
+  thk="${thk}"
+  rgba="${color}"/>
+  <xacro:u_corridor
+  name="5"
+  x="-0.5"
+  y=".5"
+  yaw="${3*PI/2}"
+  length="${L}"
+  width="${W}"
+  height="${H}"
+  thk="${thk}"
+  rgba="${color}"/>
+  <xacro:u_corridor
+  name="6"
+  x="0"
+  y="1"
+  yaw="${PI}"
+  length="${L}"
+  width="${W}"
+  height="${H}"
+  thk="${thk}"
+  rgba="${color}"/>
+  <xacro:corridor
+  name="7"
+  x="0.0"
+  y="0"
+  yaw="0"
+  length="${L}"
+  width="${W}"
+  height="${H}"
+  thk="${thk}"
+  rgba="${color}"/>
+  <xacro:corridor
   name="8"
+  x="0"
+  y="-0.5"
+  yaw="0"
+  length="${L}"
+  width="${W}"
+  height="${H}"
+  thk="${thk}"
+  rgba="${color}"/>
+  <xacro:corner
+  name="9"
+  x="0"
+  y="-1"
+  yaw="${PI}"
+  length="${L}"
+  width="${W}"
+  height="${H}"
+  thk="${thk}"
+  rgba="${color}"/>
+  <xacro:corridor
+  name="10"
+  x="-0.5"
+  y="-1"
+  yaw="${PI/2}"
+  length="${L}"
+  width="${W}"
+  height="${H}"
+  thk="${thk}"
+  rgba="${color}"/>
+  <xacro:corner
+  name="11"
   x="-1.0"
-  y="1.0"
+  y="-1"
   yaw="${0}"
   length="${L}"
@@ -538,63 +568,13 @@
   thk="${thk}"
   rgba="${color}"/>
-  <xacro:corner
-    name="9"
-    x="-1.0"
-    y="1.5"
-    yaw="${PI*3/2}"
-    length="${L}"
-    width="${W}"
-    height="${H}"
-    thk="${thk}"
-    rgba="${color}"/>
-  <xacro:corridor
-    name="10"
-    x="-1.5"
-    y="1.5"
-    yaw="${pi/2}"
-    length="${L}"
-    width="${W}"
-    height="${H}"
-    thk="${thk}"
-    rgba="${color}"/>
-  <xacro:corridor
-    name="11"
-    x="0.5"
-    y="-0.5"
-    yaw="${0}"
-    length="${L}"
-    width="${W}"
-    height="${H}"
-    thk="${thk}"
-    rgba="${color}"/>
-  <xacro:corridor
-    name="12"
-    x="0.5"
-    y="-1"
-    yaw="${0}"
-    length="${L}"
-    width="${W}"
-    height="${H}"
-    thk="${thk}"
-    rgba="${color}"/>
-  <xacro:corridor
-    name="13"
-    x="0.5"
-    y="-1.5"
-    yaw="${0}"
-    length="${L}"
-    width="${W}"
-    height="${H}"
-    thk="${thk}"
-    rgba="${color}"/>
-  <xacro:corridor
-    name="14"
-    x="0.5"
-    y="-2"
-    yaw="${0}"
-    length="${L}"
-    width="${W}"
-    height="${H}"
-    thk="${thk}"
-    rgba="${color}"/>
+  <xacro:corridor
+  name="12"
+  x="-1"
+  y="-1.5"
+  yaw="${0}"
+  length="${L}"
+  width="${W}"
+  height="${H}"
+  thk="${thk}"
+  rgba="${color}"/>
 </robot>
