Commit message: Modification pour utiliser les lidars + Readme

File: Map/Corridor/corridor.urdf (robot description, URDF)
Before this commit: robot corridor, 5 links, 4 joints
Links:
- removed link wall_e
- removed link wall_n
- removed link wall_s
- removed link wall_w
- added link -1_left, mass 0; collision box size=0.04 0.5 0.5; visual box size=0.04 0.5 0.5
- added link -1_right, mass 0; collision box size=0.04 0.5 0.5; visual box size=0.04 0.5 0.5
- added link -2_left, mass 0; collision box size=0.04 0.5 0.5; visual box size=0.04 0.5 0.5
- added link -2_right, mass 0; collision box size=0.04 0.5 0.5; visual box size=0.04 0.5 0.5
- added link 0_left, mass 0; collision box size=0.04 0.5 0.5; visual box size=0.04 0.5 0.5
- added link 0_right, mass 0; collision box size=0.04 0.5 0.5; visual box size=0.04 0.5 0.5
- added link 1_left, mass 0; collision box size=0.04 0.5 0.5; visual box size=0.04 0.5 0.5
- added link 1_right, mass 0; collision box size=0.04 0.5 0.5; visual box size=0.04 0.5 0.5
- added link Limit 1, mass 0; collision box size=0.04 3.4 1; visual box size=0.04 3.4 1
- added link Limit 2, mass 0; collision box size=0.04 3.4 1; visual box size=0.04 3.4 1
- added link Limit 3, mass 0; collision box size=0.04 4.6 1; visual box size=0.04 4.6 1
- added link Limit 4, mass 0; collision box size=0.04 4.6 1; visual box size=0.04 4.6 1
Joints:
- removed joint wall_e_world
- removed joint wall_n_world
- removed joint wall_s_world
- removed joint wall_w_world
- added joint -1_left_world: type fixed, parent world, child -1_left, origin xyz=-0.5 0.27 0 rpy=0 0 1.5707963267948966
- added joint -1_right_world: type fixed, parent world, child -1_right, origin xyz=-0.5 -0.27 0 rpy=0 0 1.5707963267948966
- added joint -2_left_world: type fixed, parent world, child -2_left, origin xyz=-1.0 0.27 0 rpy=0 0 1.5707963267948966
- added joint -2_right_world: type fixed, parent world, child -2_right, origin xyz=-1.0 -0.27 0 rpy=0 0 1.5707963267948966
- added joint 0_left_world: type fixed, parent world, child 0_left, origin xyz=1.653273178848927e-17 0.27 0 rpy=0 0 1.5707963267948966
- added joint 0_right_world: type fixed, parent world, child 0_right, origin xyz=-1.653273178848927e-17 -0.27 0 rpy=0 0 1.5707963267948966
- added joint 1_left_world: type fixed, parent world, child 1_left, origin xyz=0.5 0.27 0 rpy=0 0 1.5707963267948966
- added joint 1_right_world: type fixed, parent world, child 1_right, origin xyz=0.5 -0.27 0 rpy=0 0 1.5707963267948966
- added joint Limit 1_world: type fixed, parent world, child Limit 1, origin xyz=2.3 0 0 rpy=0 0 0
- added joint Limit 2_world: type fixed, parent world, child Limit 2, origin xyz=-2.3 0 0 rpy=0 0 0
- added joint Limit 3_world: type fixed, parent world, child Limit 3, origin xyz=0 1.7 0 rpy=0 0 1.5707963267948966
- added joint Limit 4_world: type fixed, parent world, child Limit 4, origin xyz=0 -1.7 0 rpy=0 0 1.5707963267948966

File: Map/Corridor/corridor.xacro (robot description, xacro)
@@ -9,7 +9,14 @@
   <!-- Constants -->
   <xacro:property name="PI" value="${3.141592653589793}"/>
-  <!-- Dimensions: L_in = clair-voie intérieure, L_out = dimension extérieure -->
-  <xacro:property name="L_in"  value="${CFG['length']}"/>
-  <xacro:property name="L_out" value="${CFG['length'] + 2*CFG['thk']}"/>
+  <!-- Dimensions: L = wall length -->
+  <xacro:property name="L"  value="${CFG['length']}"/>
+  <!-- Dimensions: thk = wall thikness -->
+  <xacro:property name="thk"  value="${CFG['thk']}"/>
+  <!-- Dimensions: H = wall height -->
+  <xacro:property name="H"  value="${CFG['height']}"/>
+  <!-- Dimensions: color = wall color -->
+  <xacro:property name="color"  value="${CFG['rgba']}"/>
+  <!-- Dimensions: W = corridor width -->
+  <xacro:property name="W"  value="${CFG['width']}"/>
   <!-- Wall macro -->
   <xacro:macro name="wall" params="name x y yaw length thk height rgba">
@@ -18,5 +25,5 @@
         <origin xyz="0 0 ${height/2}" rpy="0 0 0"/>
         <geometry>
-          <box size="${length} ${thk} ${height}"/>
+          <box size="${thk} ${length} ${height}"/>
         </geometry>
         <material name="${name}_mat">
@@ -27,5 +34,5 @@
         <origin xyz="0 0 ${height/2}" rpy="0 0 0"/>
         <geometry>
-          <box size="${length} ${thk} ${height}"/>
+          <box size="${thk} ${length} ${height}"/>
         </geometry>
       </collision>
@@ -41,36 +48,453 @@
     </joint>
   </xacro:macro>
+  <!-- Corridor macro -->
+  <xacro:macro name="corridor" params="name x y yaw length thk height rgba width">
+    <!-- compute rotation (cos/sin) and rotate local offsets -->
+    <xacro:property name="_yaw" value="${float(yaw)}"/>
+    <xacro:property name="_c" value="${math.cos(_yaw)}"/>
+    <xacro:property name="_s" value="${math.sin(_yaw)}"/>
+    <!-- Left wall local offset -->
+    <xacro:property name="_left_dx" value="${width/2 + thk/2}"/>
+    <xacro:property name="_left_dy" value="0"/>
+    <xacro:property name="_left_x" value="${x + _left_dx*_c - _left_dy*_s}"/>
+    <xacro:property name="_left_y" value="${y + _left_dx*_s + _left_dy*_c}"/>
+    <!-- Mur gauche -->
+    <xacro:wall
+      name="${name}_left"
+      x="${_left_x}"
+      y="${_left_y}"
+      yaw="${yaw}"
+      length="${length}"
+      thk="${thk}"
+      height="${height}"
+      rgba="${rgba}" />
+    <!-- Right wall local offset -->
+    <xacro:property name="_right_dx" value="${-(width/2 + thk/2)}"/>
+    <xacro:property name="_right_dy" value="0"/>
+    <xacro:property name="_right_x" value="${x + _right_dx*_c - _right_dy*_s}"/>
+    <xacro:property name="_right_y" value="${y + _right_dx*_s + _right_dy*_c}"/>
+    <!-- Mur droit -->
+    <xacro:wall
+      name="${name}_right"
+      x="${_right_x}"
+      y="${_right_y}"
+      yaw="${yaw}"
+      length="${length}"
+      thk="${thk}"
+      height="${height}"
+      rgba="${rgba}" />
+  </xacro:macro>
+  <!-- U_corridor macro -->
+  <xacro:macro name="u_corridor" params="name x y yaw length thk height rgba width">
+    <!-- compute rotation (cos/sin) and rotate local offsets -->
+    <xacro:property name="_yaw" value="${float(yaw)}"/>
+    <xacro:property name="_c" value="${math.cos(_yaw)}"/>
+    <xacro:property name="_s" value="${math.sin(_yaw)}"/>
+    <!-- Left wall local offset -->
+    <xacro:property name="_left_dx" value="${width/2 + thk/2}"/>
+    <xacro:property name="_left_dy" value="0"/>
+    <xacro:property name="_left_x" value="${x + _left_dx*_c - _left_dy*_s}"/>
+    <xacro:property name="_left_y" value="${y + _left_dx*_s + _left_dy*_c}"/>
+    <!-- Mur gauche -->
+    <xacro:wall
+      name="${name}_left"
+      x="${_left_x}"
+      y="${_left_y}"
+      yaw="${yaw}"
+      length="${length}"
+      thk="${thk}"
+      height="${height}"
+      rgba="${rgba}" />
+    <!-- Right wall local offset -->
+    <xacro:property name="_right_dx" value="${-(width/2 + thk/2)}"/>
+    <xacro:property name="_right_dy" value="0"/>
+    <xacro:property name="_right_x" value="${x + _right_dx*_c - _right_dy*_s}"/>
+    <xacro:property name="_right_y" value="${y + _right_dx*_s + _right_dy*_c}"/>
+    <!-- Mur droit -->
+    <xacro:wall
+      name="${name}_right"
+      x="${_right_x}"
+      y="${_right_y}"
+      yaw="${yaw}"
+      length="${length}"
+      thk="${thk}"
+      height="${height}"
+      rgba="${rgba}" />
+    <xacro:property name="_back_dx" value="0"/>
+    <xacro:property name="_back_dy" value="${-length/2-thk/2}"/>
+    <xacro:property name="_back_x" value="${x + _back_dx*_c - _back_dy*_s}"/>
+    <xacro:property name="_back_y" value="${y + _back_dx*_s + _back_dy*_c}"/>
+    <!-- Mur Derrière -->
+    <xacro:wall
+      name="${name}_back"
+      x="${_back_x}"
+      y="${_back_y}"
+      yaw="${yaw+PI/2}"
+      length="${width}"
+      thk="${thk}"
+      height="${height}"
+      rgba="${rgba}"/>
+  </xacro:macro>
+  <!-- Corner macro -->
+  <xacro:macro name="corner" params="name x y yaw length thk height rgba width">
+    <!-- compute rotation (cos/sin) and rotate local offsets -->
+    <xacro:property name="_yaw" value="${float(yaw)}"/>
+    <xacro:property name="_c" value="${math.cos(_yaw)}"/>
+    <xacro:property name="_s" value="${math.sin(_yaw)}"/>
+    <!-- Left wall local offset -->
+    <xacro:property name="_left_dx" value="${width/2 + thk/2}"/>
+    <xacro:property name="_left_dy" value="${-(length/2-width/2)/2-width/2}"/>
+    <xacro:property name="_left_x" value="${x + _left_dx*_c - _left_dy*_s}"/>
+    <xacro:property name="_left_y" value="${y + _left_dx*_s + _left_dy*_c}"/>
+    <!-- Mur Droit -->
+    <xacro:wall
+      name="${name}_left"
+      x="${_left_x}"
+      y="${_left_y}"
+      yaw="${yaw}"
+      length="${length/2-width/2}"
+      thk="${thk}"
+      height="${height}"
+      rgba="${rgba}" />
+    <!-- Right wall local offset -->
+    <xacro:property name="_right_dx" value="${-(width/2 + thk/2)}"/>
+    <xacro:property name="_right_dy" value="${-(length+width)/4+width/2}"/>
+    <xacro:property name="_right_x" value="${x + _right_dx*_c - _right_dy*_s}"/>
+    <xacro:property name="_right_y" value="${y + _right_dx*_s + _right_dy*_c}"/>
+    <!-- Mur Gauche -->
+    <xacro:wall
+      name="${name}_right"
+      x="${_right_x}"
+      y="${_right_y}"
+      yaw="${yaw}"
+      length="${(length+width)/2}"
+      thk="${thk}"
+      height="${height}"
+      rgba="${rgba}" />
+    <xacro:property name="_front_up_dx" value="${(length+width)/4-width/2}"/>
+    <xacro:property name="_front_up_dy" value="${width/2+thk/2}"/>
+    <xacro:property name="_front_up_x" value="${x + _front_up_dx*_c - _front_up_dy*_s}"/>
+    <xacro:property name="_front_up_y" value="${y + _front_up_dx*_s + _front_up_dy*_c}"/>
+    <!-- Mur Fond_haut -->
+    <xacro:wall
+      name="${name}_front_up"
+      x="${_front_up_x}"
+      y="${_front_up_y}"
+      yaw="${yaw+PI/2}"
+      length="${(length+width)/2}"
+      thk="${thk}"
+      height="${height}"
+      rgba="${rgba}"/>
+      <xacro:property name="_front_down_dx" value="${+(length/2-width/2)/2+width/2}"/>
+    <xacro:property name="_front_down_dy" value="${-width/2-thk/2}"/>
+    <xacro:property name="_front_down_x" value="${x + _front_down_dx*_c - _front_down_dy*_s}"/>
+    <xacro:property name="_front_down_y" value="${y + _front_down_dx*_s + _front_down_dy*_c}"/>
+    <!-- Mur Fond_bas -->
+    <xacro:wall
+      name="${name}_front_down"
+      x="${_front_down_x}"
+      y="${_front_down_y}"
+      yaw="${yaw+PI/2}"
+      length="${length/2-width/2}"
+      thk="${thk}"
+      height="${height}"
+      rgba="${rgba}"/>
+  </xacro:macro>
+  <!-- T macro -->
+  <xacro:macro name="T_intersection" params="name x y yaw length thk height rgba width">
+    <!-- compute rotation (cos/sin) and rotate local offsets -->
+    <xacro:property name="_yaw" value="${float(yaw)}"/>
+    <xacro:property name="_c" value="${math.cos(_yaw)}"/>
+    <xacro:property name="_s" value="${math.sin(_yaw)}"/>
+    <!-- Fond wall local offset -->
+    <xacro:property name="_left_dx" value="${0}"/>
+    <xacro:property name="_left_dy" value="${width/2+thk/2}"/>
+    <xacro:property name="_left_x" value="${x + _left_dx*_c - _left_dy*_s}"/>
+    <xacro:property name="_left_y" value="${y + _left_dx*_s + _left_dy*_c}"/>
+    <!-- Mur Fond -->
+    <xacro:wall
+      name="${name}_fond"
+      x="${_left_x}"
+      y="${_left_y}"
+      yaw="${yaw+PI/2}"
+      length="${length}"
+      thk="${thk}"
+      height="${height}"
+      rgba="${rgba}" />
+    <!-- Gauche_H wall local offset -->
+    <xacro:property name="_left_dx" value="${-(length-width)/4-width/2}"/>
+    <xacro:property name="_left_dy" value="${-width/2-thk/2}"/>
+    <xacro:property name="_left_x" value="${x + _left_dx*_c - _left_dy*_s}"/>
+    <xacro:property name="_left_y" value="${y + _left_dx*_s + _left_dy*_c}"/>
+    <!-- Mur Gauche_H -->
+    <xacro:wall
+      name="${name}_gauche_h"
+      x="${_left_x}"
+      y="${_left_y}"
+      yaw="${yaw+PI/2}"
+      length="${(length-width)/2}"
+      thk="${thk}"
+      height="${height}"
+      rgba="${rgba}" />
+    <!-- Gauche_V wall local offset -->
+    <xacro:property name="_left_dx" value="${-width/2-thk/2}"/>
+    <xacro:property name="_left_dy" value="${-(length-width)/4-width/2}"/>
+    <xacro:property name="_left_x" value="${x + _left_dx*_c - _left_dy*_s}"/>
+    <xacro:property name="_left_y" value="${y + _left_dx*_s + _left_dy*_c}"/>
+    <!-- Mur Gauche_V -->
+    <xacro:wall
+      name="${name}_gauche_v"
+      x="${_left_x}"
+      y="${_left_y}"
+      yaw="${yaw}"
+      length="${(length-width)/2}"
+      thk="${thk}"
+      height="${height}"
+      rgba="${rgba}" />
+    <!-- Droit_H wall local offset -->
+    <xacro:property name="_left_dx" value="${+(length-width)/4+width/2}"/>
+    <xacro:property name="_left_dy" value="${-width/2-thk/2}"/>
+    <xacro:property name="_left_x" value="${x + _left_dx*_c - _left_dy*_s}"/>
+    <xacro:property name="_left_y" value="${y + _left_dx*_s + _left_dy*_c}"/>
+    <!-- Mur Droit_H -->
+    <xacro:wall
+      name="${name}_droit_h"
+      x="${_left_x}"
+      y="${_left_y}"
+      yaw="${yaw+PI/2}"
+      length="${(length-width)/2}"
+      thk="${thk}"
+      height="${height}"
+      rgba="${rgba}" />
+    <!-- Droit_V wall local offset -->
+    <xacro:property name="_left_dx" value="${+width/2+thk/2}"/>
+    <xacro:property name="_left_dy" value="${-(length-width)/4-width/2}"/>
+    <xacro:property name="_left_x" value="${x + _left_dx*_c - _left_dy*_s}"/>
+    <xacro:property name="_left_y" value="${y + _left_dx*_s + _left_dy*_c}"/>
+    <!-- Mur Droit_V -->
+    <xacro:wall
+      name="${name}_droit_v"
+      x="${_left_x}"
+      y="${_left_y}"
+      yaw="${yaw}"
+      length="${(length-width)/2}"
+      thk="${thk}"
+      height="${height}"
+      rgba="${rgba}" />
+  </xacro:macro>
+  <!-- Croix macro -->
+  <xacro:macro name="C_intersection" params="name x y yaw length thk height rgba width">
+    <!-- compute rotation (cos/sin) and rotate local offsets -->
+    <xacro:property name="_yaw" value="${float(yaw)}"/>
+    <xacro:property name="_c" value="${math.cos(_yaw)}"/>
+    <xacro:property name="_s" value="${math.sin(_yaw)}"/>
+    <!-- Gauche_H wall local offset -->
+    <xacro:property name="_left_dx" value="${-(length-width)/4-width/2}"/>
+    <xacro:property name="_left_dy" value="${width/2+thk/2}"/>
+    <xacro:property name="_left_x" value="${x + _left_dx*_c - _left_dy*_s}"/>
+    <xacro:property name="_left_y" value="${y + _left_dx*_s + _left_dy*_c}"/>
+    <!-- Mur Gauche_H -->
+    <xacro:wall
+      name="${name}_gauche_h_h"
+      x="${_left_x}"
+      y="${_left_y}"
+      yaw="${yaw+PI/2}"
+      length="${(length-width)/2}"
+      thk="${thk}"
+      height="${height}"
+      rgba="${rgba}" />
+    <!-- Gauche_V wall local offset -->
+    <xacro:property name="_left_dx" value="${-width/2-thk/2}"/>
+    <xacro:property name="_left_dy" value="${(length-width)/4+width/2}"/>
+    <xacro:property name="_left_x" value="${x + _left_dx*_c - _left_dy*_s}"/>
+    <xacro:property name="_left_y" value="${y + _left_dx*_s + _left_dy*_c}"/>
+    <!-- Mur Gauche_V -->
+    <xacro:wall
+      name="${name}_gauche_v_h"
+      x="${_left_x}"
+      y="${_left_y}"
+      yaw="${yaw}"
+      length="${(length-width)/2}"
+      thk="${thk}"
+      height="${height}"
+      rgba="${rgba}" />
+    <!-- Droit_H wall local offset -->
+    <xacro:property name="_left_dx" value="${+(length-width)/4+width/2}"/>
+    <xacro:property name="_left_dy" value="${+width/2+thk/2}"/>
+    <xacro:property name="_left_x" value="${x + _left_dx*_c - _left_dy*_s}"/>
+    <xacro:property name="_left_y" value="${y + _left_dx*_s + _left_dy*_c}"/>
+    <!-- Mur Droit_H -->
+    <xacro:wall
+      name="${name}_droit_h_h"
+      x="${_left_x}"
+      y="${_left_y}"
+      yaw="${yaw+PI/2}"
+      length="${(length-width)/2}"
+      thk="${thk}"
+      height="${height}"
+      rgba="${rgba}" />
+    <!-- Droit_V wall local offset -->
+    <xacro:property name="_left_dx" value="${+width/2+thk/2}"/>
+    <xacro:property name="_left_dy" value="${+(length-width)/4+width/2}"/>
+    <xacro:property name="_left_x" value="${x + _left_dx*_c - _left_dy*_s}"/>
+    <xacro:property name="_left_y" value="${y + _left_dx*_s + _left_dy*_c}"/>
+    <!-- Mur Droit_V -->
+    <xacro:wall
+      name="${name}_droit_v_h"
+      x="${_left_x}"
+      y="${_left_y}"
+      yaw="${yaw}"
+      length="${(length-width)/2}"
+      thk="${thk}"
+      height="${height}"
+      rgba="${rgba}" />
+    <!-- Gauche_H wall local offset -->
+    <xacro:property name="_left_dx" value="${-(length-width)/4-width/2}"/>
+    <xacro:property name="_left_dy" value="${-width/2-thk/2}"/>
+    <xacro:property name="_left_x" value="${x + _left_dx*_c - _left_dy*_s}"/>
+    <xacro:property name="_left_y" value="${y + _left_dx*_s + _left_dy*_c}"/>
+    <!-- Mur Gauche_H -->
+    <xacro:wall
+      name="${name}_gauche_h"
+      x="${_left_x}"
+      y="${_left_y}"
+      yaw="${yaw+PI/2}"
+      length="${(length-width)/2}"
+      thk="${thk}"
+      height="${height}"
+      rgba="${rgba}" />
+    <!-- Gauche_V wall local offset -->
+    <xacro:property name="_left_dx" value="${-width/2-thk/2}"/>
+    <xacro:property name="_left_dy" value="${-(length-width)/4-width/2}"/>
+    <xacro:property name="_left_x" value="${x + _left_dx*_c - _left_dy*_s}"/>
+    <xacro:property name="_left_y" value="${y + _left_dx*_s + _left_dy*_c}"/>
+    <!-- Mur Gauche_V -->
+    <xacro:wall
+      name="${name}_gauche_v"
+      x="${_left_x}"
+      y="${_left_y}"
+      yaw="${yaw}"
+      length="${(length-width)/2}"
+      thk="${thk}"
+      height="${height}"
+      rgba="${rgba}" />
+    <!-- Droit_H wall local offset -->
+    <xacro:property name="_left_dx" value="${+(length-width)/4+width/2}"/>
+    <xacro:property name="_left_dy" value="${-width/2-thk/2}"/>
+    <xacro:property name="_left_x" value="${x + _left_dx*_c - _left_dy*_s}"/>
+    <xacro:property name="_left_y" value="${y + _left_dx*_s + _left_dy*_c}"/>
+    <!-- Mur Droit_H -->
+    <xacro:wall
+      name="${name}_droit_h"
+      x="${_left_x}"
+      y="${_left_y}"
+      yaw="${yaw+PI/2}"
+      length="${(length-width)/2}"
+      thk="${thk}"
+      height="${height}"
+      rgba="${rgba}" />
+    <!-- Droit_V wall local offset -->
+    <xacro:property name="_left_dx" value="${+width/2+thk/2}"/>
+    <xacro:property name="_left_dy" value="${-(length-width)/4-width/2}"/>
+    <xacro:property name="_left_x" value="${x + _left_dx*_c - _left_dy*_s}"/>
+    <xacro:property name="_left_y" value="${y + _left_dx*_s + _left_dy*_c}"/>
+    <!-- Mur Droit_V -->
+    <xacro:wall
+      name="${name}_droit_v"
+      x="${_left_x}"
+      y="${_left_y}"
+      yaw="${yaw}"
+      length="${(length-width)/2}"
+      thk="${thk}"
+      height="${height}"
+      rgba="${rgba}" />
+  </xacro:macro>
+  <!-- Map limit -->
+  <xacro:wall
+      name="Limit 1"
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