Commit message: fix pour simu fonctionnelle

File: Map/Demo_with_current_inventory/Demo_with_current_inventory.urdf (robot description, URDF)
Before this commit: robot corridor, 53 links, 52 joints
Links:
- removed link 1_back
Joints:
- removed joint 1_back_world
- joint 10_droit_h_world: origin xyz=0.25000000000000006 0.2700000000000001 0 rpy=0 0 4.71238898038469 -> xyz=-0.25 -0.27 0 rpy=0 0 1.5707963267948966
- joint 10_droit_v_world: origin xyz=0.23 0.25000000000000006 0 rpy=0 0 3.141592653589793 -> xyz=-0.22999999999999998 -0.25 0 rpy=0 0 0
- joint 10_fond_world: origin xyz=0.49999999999999994 -0.27 0 rpy=0 0 4.71238898038469 -> xyz=-0.5 0.27 0 rpy=0 0 1.5707963267948966
- joint 10_gauche_h_world: origin xyz=0.75 0.26999999999999996 0 rpy=0 0 4.71238898038469 -> xyz=-0.75 -0.27 0 rpy=0 0 1.5707963267948966
- joint 10_gauche_v_world: origin xyz=0.77 0.24999999999999997 0 rpy=0 0 3.141592653589793 -> xyz=-0.77 -0.25 0 rpy=0 0 0
- joint 11_left_world: origin xyz=1.0 0.27 0 rpy=0 0 1.5707963267948966 -> xyz=-1.0 0.27 0 rpy=0 0 1.5707963267948966
- joint 11_right_world: origin xyz=1.0 -0.27 0 rpy=0 0 1.5707963267948966 -> xyz=-1.0 -0.27 0 rpy=0 0 1.5707963267948966
- joint 12_back_world: origin xyz=1.77 -1.653273178848927e-17 0 rpy=0 0 3.141592653589793 -> xyz=-1.77 4.9598195365467806e-17 0 rpy=0 0 6.283185307179586
- joint 12_left_world: origin xyz=1.5 0.27 0 rpy=0 0 1.5707963267948966 -> xyz=-1.5 -0.27 0 rpy=0 0 4.71238898038469
- joint 12_right_world: origin xyz=1.5 -0.27 0 rpy=0 0 1.5707963267948966 -> xyz=-1.5 0.27 0 rpy=0 0 4.71238898038469
- joint 13_left_world: origin xyz=0.77 0.5 0 rpy=0 0 0 -> xyz=-0.22999999999999998 -0.5 0 rpy=0 0 0
- joint 13_right_world: origin xyz=0.22999999999999998 0.5 0 rpy=0 0 0 -> xyz=-0.77 -0.5 0 rpy=0 0 0
- joint 14_front_down_world: origin xyz=0.75 0.73 0 rpy=0 0 1.5707963267948966 -> xyz=-0.75 -0.73 0 rpy=0 0 4.71238898038469
- joint 14_front_up_world: origin xyz=0.5 1.27 0 rpy=0 0 1.5707963267948966 -> xyz=-0.5 -1.27 0 rpy=0 0 4.71238898038469
- joint 14_left_world: origin xyz=0.77 0.75 0 rpy=0 0 0 -> xyz=-0.77 -0.75 0 rpy=0 0 3.141592653589793
- joint 14_right_world: origin xyz=0.22999999999999998 1.0 0 rpy=0 0 0 -> xyz=-0.22999999999999998 -1.0 0 rpy=0 0 3.141592653589793
- joint 15_left_world: origin xyz=1.0 1.27 0 rpy=0 0 1.5707963267948966 -> xyz=-1.0 -0.73 0 rpy=0 0 1.5707963267948966
- joint 15_right_world: origin xyz=1.0 0.73 0 rpy=0 0 1.5707963267948966 -> xyz=-1.0 -1.27 0 rpy=0 0 1.5707963267948966
- joint 16_left_world: origin xyz=1.5 1.27 0 rpy=0 0 1.5707963267948966 -> xyz=-1.5 -0.73 0 rpy=0 0 1.5707963267948966
- joint 16_right_world: origin xyz=1.5 0.73 0 rpy=0 0 1.5707963267948966 -> xyz=-1.5 -1.27 0 rpy=0 0 1.5707963267948966
- joint 17_back_world: origin xyz=2.27 1.0 0 rpy=0 0 3.141592653589793 -> xyz=-2.27 -1.0 0 rpy=0 0 6.283185307179586
- joint 17_left_world: origin xyz=2.0 1.27 0 rpy=0 0 1.5707963267948966 -> xyz=-2.0 -1.27 0 rpy=0 0 4.71238898038469
- joint 17_right_world: origin xyz=2.0 0.73 0 rpy=0 0 1.5707963267948966 -> xyz=-2.0 -0.73 0 rpy=0 0 4.71238898038469
- joint 1_left_world: origin xyz=-1.77 0.5 0 rpy=0 0 3.141592653589793 -> xyz=1.77 -0.5 0 rpy=0 0 0
- joint 1_right_world: origin xyz=-1.23 0.49999999999999994 0 rpy=0 0 3.141592653589793 -> xyz=1.23 -0.5 0 rpy=0 0 0
- joint 2_left_world: origin xyz=-1.23 0.0 0 rpy=0 0 0 -> xyz=1.77 0.0 0 rpy=0 0 0
- joint 2_right_world: origin xyz=-1.77 0.0 0 rpy=0 0 0 -> xyz=1.23 0.0 0 rpy=0 0 0
- joint 3_left_world: origin xyz=-1.23 -0.5 0 rpy=0 0 0 -> xyz=1.77 0.5 0 rpy=0 0 0
- joint 3_right_world: origin xyz=-1.77 -0.5 0 rpy=0 0 0 -> xyz=1.23 0.5 0 rpy=0 0 0
- joint 4_front_down_world: origin xyz=-1.23 -0.75 0 rpy=0 0 3.141592653589793 -> xyz=1.23 0.75 0 rpy=0 0 6.283185307179586
- joint 4_front_up_world: origin xyz=-1.77 -1.0 0 rpy=0 0 3.141592653589793 -> xyz=1.77 1.0 0 rpy=0 0 6.283185307179586
- joint 4_left_world: origin xyz=-1.25 -0.73 0 rpy=0 0 1.5707963267948966 -> xyz=1.25 0.73 0 rpy=0 0 4.71238898038469
- joint 4_right_world: origin xyz=-1.5 -1.27 0 rpy=0 0 1.5707963267948966 -> xyz=1.5 1.27 0 rpy=0 0 4.71238898038469
- joint 5_left_world: origin xyz=-1.0 -0.73 0 rpy=0 0 1.5707963267948966 -> xyz=1.0 1.27 0 rpy=0 0 1.5707963267948966
- joint 5_right_world: origin xyz=-1.0 -1.27 0 rpy=0 0 1.5707963267948966 -> xyz=1.0 0.73 0 rpy=0 0 1.5707963267948966
- joint 6_front_down_world: origin xyz=-0.75 -0.73 0 rpy=0 0 4.71238898038469 -> xyz=0.75 0.73 0 rpy=0 0 1.5707963267948966
- joint 6_front_up_world: origin xyz=-0.5 -1.27 0 rpy=0 0 4.71238898038469 -> xyz=0.5 1.27 0 rpy=0 0 1.5707963267948966
- joint 6_left_world: origin xyz=-0.77 -0.75 0 rpy=0 0 3.141592653589793 -> xyz=0.77 0.75 0 rpy=0 0 0
- joint 6_right_world: origin xyz=-0.22999999999999998 -1.0 0 rpy=0 0 3.141592653589793 -> xyz=0.22999999999999998 1.0 0 rpy=0 0 0
- joint 7_left_world: origin xyz=-0.22999999999999998 -0.5 0 rpy=0 0 0 -> xyz=0.77 0.5 0 rpy=0 0 0
- joint 7_right_world: origin xyz=-0.77 -0.5 0 rpy=0 0 0 -> xyz=0.22999999999999998 0.5 0 rpy=0 0 0
- joint 8_front_down_world: origin xyz=-0.25 -0.27 0 rpy=0 0 1.5707963267948966 -> xyz=0.25000000000000006 0.2700000000000001 0 rpy=0 0 4.71238898038469
- joint 8_front_up_world: origin xyz=-0.5 0.27 0 rpy=0 0 1.5707963267948966 -> xyz=0.49999999999999994 -0.27 0 rpy=0 0 4.71238898038469
- joint 8_left_world: origin xyz=-0.22999999999999998 -0.25 0 rpy=0 0 0 -> xyz=0.23 0.25000000000000006 0 rpy=0 0 3.141592653589793
- joint 8_right_world: origin xyz=-0.77 0.0 0 rpy=0 0 0 -> xyz=0.77 -3.306546357697854e-17 0 rpy=0 0 3.141592653589793

File: Map/Demo_with_current_inventory/Demo_with_current_inventory.xacro (robot description, xacro)
@@ -448,9 +448,9 @@
       rgba="${color}"/>
   <!-- corridors (positionnés pour que l'intérieur fasse width) -->
-  <xacro:u_corridor
+  <xacro:corridor
   name="1"
-  x="2"
+  x="1.5"
   y="-0.5"
-  yaw="${PI}"
+  yaw="${0}"
   length="0.5"
   thk="0.04"
@@ -460,5 +460,5 @@
   <xacro:corridor
   name="2"
-  x="2"
+  x="1.5"
   y="0"
   yaw="${0}"
@@ -470,5 +470,5 @@
   <xacro:corridor
   name="3"
-  x="2"
+  x="1.5"
   y="0.5"
   yaw="${0}"
@@ -480,7 +480,7 @@
   <xacro:corner
   name="4"
-  x="2"
+  x="1.5"
   y="1"
-  yaw="${PI/2}"
+  yaw="${3*PI/2}"
   length="${L}"
   width="${W}"
@@ -491,5 +491,5 @@
   name="5"
   x="1"
-  y="1.5"
+  y="1"
   yaw="${PI/2}"
   length="${L}"
@@ -502,5 +502,5 @@
   x="0.5"
   y="1"
-  yaw="${PI}"
+  yaw="${0}"
   length="${L}"
   width="${W}"
@@ -522,5 +522,5 @@
   x="0.5"
   y="0"
-  yaw="${0}"
+  yaw="${PI}"
   length="${L}"
   width="${W}"
@@ -540,7 +540,7 @@
   <xacro:T_intersection
   name="10"
-  x="0.5"
+  x="-0.5"
   y="0"
-  yaw="${PI}"
+  yaw="${0}"
   length="${L}"
   width="${W}"
@@ -550,5 +550,5 @@
   <xacro:corridor
   name="11"
-  x="1"
+  x="-1"
   y="0"
   yaw="${PI/2}"
@@ -560,7 +560,7 @@
   <xacro:u_corridor
   name="12"
-  x="1.5"
+  x="-1.5"
   y="0"
-  yaw="${PI/2}"
+  yaw="${3*PI/2}"
   length="0.5"
   thk="0.04"
@@ -570,6 +570,6 @@
   <xacro:corridor
   name="13"
-  x="0.5"
-  y="0.5"
+  x="-0.5"
+  y="-0.5"
   yaw="${0}"
   length="${L}"
@@ -580,7 +580,7 @@
   <xacro:corner
   name="14"
-  x="0.5"
-  y="1"
-  yaw="${0}"
+  x="-0.5"
+  y="-1"
+  yaw="${PI}"
   length="${L}"
   width="${W}"
@@ -590,6 +590,6 @@
   <xacro:corridor
   name="15"
-  x="1"
-  y="1"
+  x="-1"
+  y="-1"
   yaw="${PI/2}"
   length="${L}"
@@ -600,6 +600,6 @@
   <xacro:corridor
   name="16"
-  x="1.5"
-  y="1"
+  x="-1.5"
+  y="-1"
   yaw="${PI/2}"
   length="${L}"
@@ -610,7 +610,7 @@
   <xacro:u_corridor
   name="17"
-  x="2"
-  y="1"
-  yaw="${PI/2}"
+  x="-2"
+  y="-1"
+  yaw="${3*PI/2}"
   length="0.5"
   thk="0.04"
